File: Electronics/TestTarget/TestTarget.kicad_pcb (KiCad board)
At the start: 2 copper layers, 8 parts, among them IC1 ATTINY13A-P, P1 CONN_02X03

Commit message: ... What was I doing :S
Parts:
- added BT1: Battery, Pin_Headers:Pin_Header_Straight_1x02, F.Cu at (139.7, 97.8)
- added D3: LED-G, LEDs:LED-3MM, F.Cu at (157.5, 85.1)
- added D4: D, Discret:R1, F.Cu at (142.2, 94.0)
- added R5: 5KΩ, Discret:R1, F.Cu at (158.8, 87.6)
- added SW1: SPST, Pin_Headers:Pin_Header_Straight_1x03, F.Cu at (139.7, 95.2)
- D2: footprint Discret:D3 -> Discret:R1
- R1, R2, R3: value 230Ω -> 470Ω
- moved R3 39.4 mm to (156.2, 92.7)
- moved R2 39.4 mm to (156.2, 90.2)
- moved IC1 34.3 mm to (144.8, 90.2)
- moved P1 34.3 mm to (144.8, 85.1)
- moved R4 34.3 mm to (142.2, 88.9)
- moved D2 31.8 mm to (142.2, 83.8), turned to 270 degrees
- moved R1 29.2 mm to (156.2, 97.8)
- moved D1 26.7 mm to (160.0, 97.8), turned to 180 degrees
