File: Electronics/MainBoard/MainBoard.sch (KiCad schematic (older format))
At the start: 18 parts, among them CN1 RCable_Con_Front, CN2 RCable_Con_Front, Q1 Q_PNP_CBE, U1 LT1004_1.2V

Commit message: More work on the electronics scematics, slowly starting to get the hang of it.
Parts:
- added CN3: RCable_Con_VEST, Pin_Headers:Pin_Header_Angled_2x05, symbol RCable_Con_VEST
- added M1: Vibr_Motor, Wire_Pads:SolderWirePad_2x_0-8mmDrill, symbol Vibr_Motor
- added R7: 68kΩ, Discret:R1, symbol R
- added R8: 33kΩ, Discret:R1, symbol R
- added SP1: SPEAKER, Buzzers_Beepers:BUZZER, symbol SPEAKER
- added SW1: SW_PUSH, Buttons_Switches_ThroughHole:SW_PUSH_SMALL, symbol SW_PUSH
- added SW2: SPST, Buttons_Switches_ThroughHole:SW_DIP_x1_Slide, symbol SPST
- BT1: footprint (none) -> Wire_Pads:SolderWirePad_2x_1-5mmDrill
- C1, C2: footprint (none) -> Capacitors_ThroughHole:C_Disc_D3_P2.5
- CN1: renamed from CN2; footprint (none) -> Pin_Headers:Pin_Header_Straight_2x05
- CN2: renamed from CN1; footprint (none) -> Pin_Headers:Pin_Header_Straight_2x05
- D1: footprint (none) -> LEDs:LED-3MM
- D2: footprint (none) -> LEDs:LED-RGB-5MM_Common_Cathode
- MCU1: footprint DIL28 -> Housings_DIP:DIP-28_W7.62mm
- Q1, U1: footprint (none) -> TO_SOT_Packages_THT:TO-92_Inline_Wide
- QRZ1: footprint (none) -> Crystals:Crystal_HC49-U_Vertical
- R1, R2, R3, R4, R5, R6: footprint (none) -> Discret:R1
- SPI1: footprint (none) -> Pin_Headers:Pin_Header_Angled_2x03
Connections:
- net labels added: BZR, B_LED, G_LED, IR_IN, IR_LED, R_LED, TRG, VBR, V_SENS
- net labels removed: +3V3, +5V
- wire segments 63 -> 93
Other:
- moved on the sheet: BT1

Commit message: Hopefully developed the final version of the prototype electronics.
Parts:
- BT1: footprint Wire_Pads:SolderWirePad_2x_1-5mmDrill -> Main-Cache:SolderWirePad_2x_0-8mmDrill
- M1: footprint Wire_Pads:SolderWirePad_2x_0-8mmDrill -> Main-Cache:SolderWirePad_2x_0-8mmDrill
- SW1: footprint Buttons_Switches_ThroughHole:SW_PUSH_SMALL -> Main-Cache:SolderWirePad_2x_0-8mmDrill
Changed lines of the file:
@@
 F 0 "MCU1" H 5350 4800 50  0000 L BNN
 F 1 "ATMEGA328P-P" H 6500 2150 50  0000 L BNN
-F 2 "Housings_DIP:DIP-28_W7.62mm" H 6100 3550 50  0000 C CIN
+F 2 "Housings_DIP:DIP-28_W7.62mm" H 6100 3550 50  0001 C CIN
 F 3 "" H 6100 3550 50  0000 C CNN
 	1    6100 3550
@@
 	8550 3200 8550 3300
 $Comp
-L GND #PWR14
+L GND #PWR01
 U 1 1 572B3BB9
 P 8550 3300
-F 0 "#PWR14" H 8550 3050 50  0001 C CNN
+F 0 "#PWR01" H 8550 3050 50  0001 C CNN
 F 1 "GND" H 8550 3150 50  0000 C CNN
 F 2 "" H 8550 3300 50  0000 C CNN
@@
 Connection ~ 8100 3200
 $Comp
-L GND #PWR3
+L GND #PWR02
 U 1 1 572B3ED7
 P 5200 4800
-F 0 "#PWR3" H 5200 4550 50  0001 C CNN
+F 0 "#PWR02" H 5200 4550 50  0001 C CNN
 F 1 "GND" H 5200 4650 50  0000 C CNN
 F 2 "" H 5200 4800 50  0000 C CNN
@@
 	5200 2750 5200 2450
 $Comp
-L GND #PWR1
+L GND #PWR03
 U 1 1 572B4A46
 P 4900 3350
-F 0 "#PWR1" H 4900 3100 50  0001 C CNN
+F 0 "#PWR03" H 4900 3100 50  0001 C CNN
 F 1 "GND" H 4900 3200 50  0000 C CNN
 F 2 "" H 4900 3350 50  0000 C CNN
@@
 F 0 "BT1" H 10350 5750 50  0000 L CNN
 F 1 "Battery" H 10350 5650 50  0000 L CNN
-F 2 "Wire_Pads:SolderWirePad_2x_1-5mmDrill" V 10250 5740 50  0001 C CNN
+F 2 "Main-Cache:SolderWirePad_2x_0-8mmDrill" V 10250 5740 50  0001 C CNN
 F 3 "" V 10250 5740 50  0000 C CNN
 	1    10250 5700
@@
 $EndComp
 $Comp
-L GND #PWR16
+L GND #PWR04
 U 1 1 572B59E3
 P 10250 5850
-F 0 "#PWR16" H 10250 5600 50  0001 C CNN
+F 0 "#PWR04" H 10250 5600 50  0001 C CNN
 F 1 "GND" H 10250 5700 50  0000 C CNN
 F 2 "" H 10250 5850 50  0000 C CNN
@@
 $EndComp
 $Comp
-L +3.3V #PWR12
+L +3.3V #PWR05
 U 1 1 572B6CF2
 P 8500 1450
-F 0 "#PWR12" H 8500 1300 50  0001 C CNN
+F 0 "#PWR05" H 8500 1300 50  0001 C CNN
 F 1 "+3.3V" H 8500 1590 50  0000 C CNN
 F 2 "" H 8500 1450 50  0000 C CNN
@@
 $EndComp
 $Comp
-L +3.3V #PWR15
+L +3.3V #PWR06
 U 1 1 572B6F24
 P 10250 4550
-F 0 "#PWR15" H 10250 4400 50  0001 C CNN
+F 0 "#PWR06" H 10250 4400 50  0001 C CNN
 F 1 "+3.3V" H 10250 4690 50  0000 C CNN
 F 2 "" H 10250 4550 50  0000 C CNN
@@
 $EndComp
 $Comp
-L +3.3V #PWR2
+L +3.3V #PWR07
 U 1 1 572B7083
 P 5200 2450
-F 0 "#PWR2" H 5200 2300 50  0001 C CNN
+F 0 "#PWR07" H 5200 2300 50  0001 C CNN
 F 1 "+3.3V" H 5200 2590 50  0000 C CNN
 F 2 "" H 5200 2450 50  0000 C CNN
@@
 	1800 3000 1900 3000
 $Comp
-L GND #PWR10
+L GND #PWR08
 U 1 1 572D7F60
 P 8300 3600
-F 0 "#PWR10" H 8300 3350 50  0001 C CNN
+F 0 "#PWR08" H 8300 3350 50  0001 C CNN
 F 1 "GND" H 8300 3450 50  0000 C CNN
 F 2 "" H 8300 3600 50  0000 C CNN
@@
 	8400 3600 8300 3600
 $Comp
-L +3.3V #PWR8
+L +3.3V #PWR09
 U 1 1 572D9157
 P 8100 3800
-F 0 "#PWR8" H 8100 3650 50  0001 C CNN
+F 0 "#PWR09" H 8100 3650 50  0001 C CNN
 F 1 "+3.3V" H 8100 3940 50  0000 C CNN
 F 2 "" H 8100 3800 50  0000 C CNN
@@
 $EndComp
 $Comp
-L +3.3V #PWR7
+L +3.3V #PWR010
 U 1 1 572DCEA7
 P 7950 2050
-F 0 "#PWR7" H 7950 1900 50  0001 C CNN
+F 0 "#PWR010" H 7950 1900 50  0001 C CNN
 F 1 "+3.3V" H 7950 2190 50  0000 C CNN
 F 2 "" H 7950 2050 50  0000 C CNN
@@
 $EndComp
 $Comp
-L GND #PWR6
+L GND #PWR011
 U 1 1 572CF9FB
 P 7150 1950
-F 0 "#PWR6" H 7150 1700 50  0001 C CNN
+F 0 "#PWR011" H 7150 1700 50  0001 C CNN
 F 1 "GND" H 7150 1800 50  0000 C CNN
 F 2 "" H 7150 1950 50  0000 C CNN
@@
 $EndComp
 $Comp
-L +3.3V #PWR5
+L +3.3V #PWR012
 U 1 1 572CFBB3
 P 7150 1350
-F 0 "#PWR5" H 7150 1200 50  0001 C CNN
+F 0 "#PWR012" H 7150 1200 50  0001 C CNN
 F 1 "+3.3V" H 7150 1490 50  0000 C CNN
 F 2 "" H 7150 1350 50  0000 C CNN
@@
 SCL
 $Comp
-L GND #PWR11
+L GND #PWR013
 U 1 1 572D931B
 P 8300 4750
-F 0 "#PWR11" H 8300 4500 50  0001 C CNN
+F 0 "#PWR013" H 8300 4500 50  0001 C CNN
 F 1 "GND" H 8300 4600 50  0000 C CNN
 F 2 "" H 8300 4750 50  0000 C CNN
@@
 	8400 4750 8300 4750
 $Comp
-L +3.3V #PWR9
+L +3.3V #PWR014
 U 1 1 572D98DD
 P 8100 5000
-F 0 "#PWR9" H 8100 4850 50  0001 C CNN
+F 0 "#PWR014" H 8100 4850 50  0001 C CNN
 F 1 "+3.3V" H 8100 5140 50  0000 C CNN
 F 2 "" H 8100 5000 50  0000 C CNN
@@
 F 0 "SW1" H 5950 6010 50  0000 C CNN
 F 1 "SW_PUSH" H 5800 5820 50  0000 C CNN
-F 2 "Buttons_Switches_ThroughHole:SW_PUSH_SMALL" H 5800 5900 50  0001 C CNN
+F 2 "Main-Cache:SolderWirePad_2x_0-8mmDrill" H 5800 5900 50  0001 C CNN
 F 3 "" H 5800 5900 50  0000 C CNN
 	1    5800 5900
@@
 F 0 "M1" H 6350 6350 60  0000 C CNN
 F 1 "Vibr_Motor" H 6150 6450 60  0000 C CNN
-F 2 "Wire_Pads:SolderWirePad_2x_0-8mmDrill" H 6000 6400 60  0001 C CNN
+F 2 "Main-Cache:SolderWirePad_2x_0-8mmDrill" H 6000 6400 60  0001 C CNN
 F 3 "" H 6000 6400 60  0000 C CNN
 	1    6100 6400
@@
 Connection ~ 5450 6350
 $Comp
-L GND #PWR4
+L GND #PWR015
 U 1 1 572E5080
 P 5450 6400
-F 0 "#PWR4" H 5450 6150 50  0001 C CNN
+F 0 "#PWR015" H 5450 6150 50  0001 C CNN
 F 1 "GND" H 5450 6250 50  0000 C CNN
 F 2 "" H 5450 6400 50  0000 C CNN
@@
 VBR
 $Comp
-L GND #PWR13
+L GND #PWR016
 U 1 1 572EF82E
 P 8500 1650
-F 0 "#PWR13" H 8500 1400 50  0001 C CNN
+F 0 "#PWR016" H 8500 1400 50  0001 C CNN
 F 1 "GND" H 8500 1500 50  0000 C CNN
 F 2 "" H 8500 1650 50  0000 C CNN

Commit message: First implementation of the eclipse code, as well as some slight further changes to the electronics board.
Parts:
- added D3: D, Discret:R1, symbol D
- R1: value 50KΩ -> 47KΩ
- R2: value 14Ω -> 10Ω
- R7: value 68kΩ -> 47kΩ
- R8: value 33kΩ -> 22kΩ
Connections:
- net at BT1.1: now also D3.2 (A); no longer SW2.1
- new net: D3.1 (K), SW2.1
Other:
- moved on the sheet: SW2
Changed lines of the file:
@@
 P 4900 2900
 F 0 "R1" V 4980 2900 50  0000 C CNN
-F 1 "50KΩ" V 4900 2900 50  0000 C CNN
+F 1 "47KΩ" V 4900 2900 50  0000 C CNN
 F 2 "Discret:R1" V 4830 2900 50  0001 C CNN
 F 3 "" H 4900 2900 50  0000 C CNN
@@
 P 1350 1700
 F 0 "R2" V 1430 1700 50  0000 C CNN
-F 1 "14Ω" V 1350 1700 50  0000 C CNN
+F 1 "10Ω" V 1350 1700 50  0000 C CNN
 F 2 "Discret:R1" V 1280 1700 50  0001 C CNN
 F 3 "" H 1350 1700 50  0000 C CNN
@@
 L +3.3V #PWR06
 U 1 1 572B6F24
-P 10250 4550
-F 0 "#PWR06" H 10250 4400 50  0001 C CNN
-F 1 "+3.3V" H 10250 4690 50  0000 C CNN
-F 2 "" H 10250 4550 50  0000 C CNN
-F 3 "" H 10250 4550 50  0000 C CNN
-	1    10250 4550
+P 10250 4250
+F 0 "#PWR06" H 10250 4100 50  0001 C CNN
+F 1 "+3.3V" H 10250 4390 50  0000 C CNN
+F 2 "" H 10250 4250 50  0000 C CNN
+F 3 "" H 10250 4250 50  0000 C CNN
+	1    10250 4250
 	1    0    0    -1
 $EndComp
@@
 P 7150 1500
 F 0 "R7" V 7230 1500 50  0000 C CNN
-F 1 "68kΩ" V 7150 1500 50  0000 C CNN
+F 1 "47kΩ" V 7150 1500 50  0000 C CNN
 F 2 "Discret:R1" V 7080 1500 50  0001 C CNN
 F 3 "" H 7150 1500 50  0000 C CNN
@@
 P 7150 1800
 F 0 "R8" V 7230 1800 50  0000 C CNN
-F 1 "33kΩ" V 7150 1800 50  0000 C CNN
+F 1 "22kΩ" V 7150 1800 50  0000 C CNN
 F 2 "Discret:R1" V 7080 1800 50  0001 C CNN
 F 3 "" H 7150 1800 50  0000 C CNN
@@
 L SPST SW2
 U 1 1 572DFDFF
-P 10250 5050
-F 0 "SW2" H 10250 5150 50  0000 C CNN
-F 1 "SPST" H 10250 4950 50  0000 C CNN
-F 2 "Buttons_Switches_ThroughHole:SW_DIP_x1_Slide" H 10250 5050 50  0001 C CNN
-F 3 "" H 10250 5050 50  0000 C CNN
-	1    10250 5050
+P 10250 4750
+F 0 "SW2" H 10250 4850 50  0000 C CNN
+F 1 "SPST" H 10250 4650 50  0000 C CNN
+F 2 "Buttons_Switches_ThroughHole:SW_DIP_x1_Slide" H 10250 4750 50  0001 C CNN
+F 3 "" H 10250 4750 50  0000 C CNN
+	1    10250 4750
 	0    -1   -1   0
 $EndComp
@@
 	1    0    0    -1
 $EndComp
+$Comp
+L D D3
+U 1 1 572DFB0F
+P 10250 5400
+F 0 "D3" H 10250 5500 50  0000 C CNN
+F 1 "D" H 10250 5300 50  0000 C CNN
+F 2 "Discret:R1" H 10250 5400 50  0001 C CNN
+F 3 "" H 10250 5400 50  0000 C CNN
+	1    10250 5400
+	0    1    1    0
+$EndComp
 $EndSCHEMATC

Commit message: Adjusted electronics for new knowledge :3
Parts:
- removed R1: 47KΩ, Discret:R1, symbol R
- removed R2: 10Ω, Discret:R1, symbol R
- removed U1: LT1004_1.2V, TO_SOT_Packages_THT:TO-92_Inline_Wide, symbol LT1004_1.2V
- added C3: 22uF, Capacitors_ThroughHole:CP_Radial_D5.0mm_P2.50mm, symbol C
- added C?: 22uF, symbol C
- added J1: CONN_02X04, Pin_Headers:Pin_Header_Straight_2x04_Pitch2.54mm, symbol CONN_02X04
- added R10, R11, R9: RST, Resistors_ThroughHole:R_Axial_DIN0204_L3.6mm_D1.6mm_P2.54mm_Vertical, symbol R_Small
- BT1: symbol Battery -> Battery-RESCUE-MainBoard
- D1: symbol LED -> LED-RESCUE-MainBoard
- D2: symbol LED_RCBG -> LED_RCBG-RESCUE-MainBoard
Connections:
- net +3V3: now also J1.7 (P7), R10.2, R11.1, R9.1
- net GND: now also C3.2, J1.2 (P2)
- net IR_IN: now also MCU1.14 ((PCINT0/CLKO/ICP1)PB0); no longer MCU1.13 ((PCINT23/AIN1)PD7)
- net SCL: now also J1.4 (P4)
- net SDA: now also J1.1 (P1)
- net at MCU1.21 (AREF): now also C3.1
- net at D1.2 (A): now also CN2.2 (Vcc), C?.1
- net at CN2.1 (GND), D2.2 (COMMON_CATHODE), Q1.1 (C): now also C?.2
- new net: J1.3 (P3), R11.2
- new net: J1.5 (P5), R9.2
- new net: J1.6 (P6), R10.1
- new net HIT_REC: J1.8 (P8)
Other:
- note added: "GPIO 01"
- note added: "GPIO 02"
- note added: "GPIO 03"
Changed lines of the file:
@@
 EESchema Schematic File Version 2
+LIBS:MainBoard-rescue
 LIBS:power
 LIBS:device
@@
 	4900 3050 5200 3050
 Wire Wire Line
-	4900 2750 5200 2750
-Wire Wire Line
 	5200 2750 5200 2450
 $Comp
-L GND #PWR03
-U 1 1 572B4A46
-P 4900 3350
-F 0 "#PWR03" H 4900 3100 50  0001 C CNN
-F 1 "GND" H 4900 3200 50  0000 C CNN
-F 2 "" H 4900 3350 50  0000 C CNN
-F 3 "" H 4900 3350 50  0000 C CNN
-	1    4900 3350
-	1    0    0    -1
-$EndComp
-$Comp
-L R R1
-U 1 1 572B4D75
-P 4900 2900
-F 0 "R1" V 4980 2900 50  0000 C CNN
-F 1 "47KΩ" V 4900 2900 50  0000 C CNN
-F 2 "Discret:R1" V 4830 2900 50  0001 C CNN
-F 3 "" H 4900 2900 50  0000 C CNN
-	1    4900 2900
-	1    0    0    -1
-$EndComp
-$Comp
-L LT1004_1.2V U1
-U 1 1 572B4E8D
-P 4900 3200
-F 0 "U1" H 4900 3300 50  0000 C CNN
-F 1 "LT1004_1.2V" H 4900 3100 50  0000 C CNN
-F 2 "TO_SOT_Packages_THT:TO-92_Inline_Wide" H 4900 3200 50  0001 C CNN
-F 3 "" H 4900 3200 50  0000 C CNN
-	1    4900 3200
-	0    1    1    0
-$EndComp
-$Comp
-L Battery BT1
+L Battery-RESCUE-MainBoard BT1
 U 1 1 572B5519
 P 10250 5700
@@
 $EndComp
 $Comp
-L GND #PWR04
+L GND #PWR03
 U 1 1 572B59E3
 P 10250 5850
-F 0 "#PWR04" H 10250 5600 50  0001 C CNN
+F 0 "#PWR03" H 10250 5600 50  0001 C CNN
 F 1 "GND" H 10250 5700 50  0000 C CNN
 F 2 "" H 10250 5850 50  0000 C CNN
@@
 NoConn ~ 7500 3100
 $Comp
-L LED D1
+L LED-RESCUE-MainBoard D1
 U 1 1 572B5B25
 P 1200 1900
@@
 $EndComp
 $Comp
-L R R2
-U 1 1 572B617E
-P 1350 1700
-F 0 "R2" V 1430 1700 50  0000 C CNN
-F 1 "10Ω" V 1350 1700 50  0000 C CNN
-F 2 "Discret:R1" V 1280 1700 50  0001 C CNN
-F 3 "" H 1350 1700 50  0000 C CNN
-	1    1350 1700
-	0    1    1    0
-$EndComp
-$Comp
-L +3.3V #PWR05
+L +3.3V #PWR04
 U 1 1 572B6CF2
 P 8500 1450
-F 0 "#PWR05" H 8500 1300 50  0001 C CNN
+F 0 "#PWR04" H 8500 1300 50  0001 C CNN
 F 1 "+3.3V" H 8500 1590 50  0000 C CNN
 F 2 "" H 8500 1450 50  0000 C CNN
@@
 $EndComp
 $Comp
-L +3.3V #PWR06
+L +3.3V #PWR05
 U 1 1 572B6F24
 P 10250 4250
-F 0 "#PWR06" H 10250 4100 50  0001 C CNN
+F 0 "#PWR05" H 10250 4100 50  0001 C CNN
 F 1 "+3.3V" H 10250 4390 50  0000 C CNN
 F 2 "" H 10250 4250 50  0000 C CNN
@@
 $EndComp
 $Comp
-L +3.3V #PWR07
+L +3.3V #PWR06
 U 1 1 572B7083
 P 5200 2450
-F 0 "#PWR07" H 5200 2300 50  0001 C CNN
+F 0 "#PWR06" H 5200 2300 50  0001 C CNN
 F 1 "+3.3V" H 5200 2590 50  0000 C CNN
 F 2 "" H 5200 2450 50  0000 C CNN
@@
 $EndComp
 $Comp
-L LED_RCBG D2
+L LED_RCBG-RESCUE-MainBoard D2
 U 1 1 572B7C1A
 P 1500 2800
@@
 	1800 3000 1900 3000
 $Comp
-L GND #PWR08
+L GND #PWR07
 U 1 1 572D7F60
 P 8300 3600
-F 0 "#PWR08" H 8300 3350 50  0001 C CNN
+F 0 "#PWR07" H 8300 3350 50  0001 C CNN
 F 1 "GND" H 8300 3450 50  0000 C CNN
 F 2 "" H 8300 3600 50  0000 C CNN
@@
 	8400 3600 8300 3600
 $Comp
-L +3.3V #PWR09
+L +3.3V #PWR08
 U 1 1 572D9157
 P 8100 3800
-F 0 "#PWR09" H 8100 3650 50  0001 C CNN
+F 0 "#PWR08" H 8100 3650 50  0001 C CNN
 F 1 "+3.3V" H 8100 3940 50  0000 C CNN
 F 2 "" H 8100 3800 50  0000 C CNN
@@
 $EndComp
 $Comp
-L +3.3V #PWR010
+L +3.3V #PWR09
 U 1 1 572DCEA7
 P 7950 2050
-F 0 "#PWR010" H 7950 1900 50  0001 C CNN
+F 0 "#PWR09" H 7950 1900 50  0001 C CNN
 F 1 "+3.3V" H 7950 2190 50  0000 C CNN
 F 2 "" H 7950 2050 50  0000 C CNN
@@
 	1500 2300 2450 2300
 Wire Wire Line
-	2450 2100 2400 2100
+	2400 2100 2450 2100
 Wire Wire Line
 	1700 2200 1500 2000
@@
 $EndComp
 $Comp
-L GND #PWR011
+L GND #PWR010
 U 1 1 572CF9FB
 P 7150 1950
-F 0 "#PWR011" H 7150 1700 50  0001 C CNN
+F 0 "#PWR010" H 7150 1700 50  0001 C CNN
 F 1 "GND" H 7150 1800 50  0000 C CNN
 F 2 "" H 7150 1950 50  0000 C CNN
@@
 $EndComp
 $Comp
-L +3.3V #PWR012
+L +3.3V #PWR011
 U 1 1 572CFBB3
 P 7150 1350
-F 0 "#PWR012" H 7150 1200 50  0001 C CNN
+F 0 "#PWR011" H 7150 1200 50  0001 C CNN
 F 1 "+3.3V" H 7150 1490 50  0000 C CNN
 F 2 "" H 7150 1350 50  0000 C CNN
@@
 SCL
 $Comp
-L GND #PWR013
+L GND #PWR012
 U 1 1 572D931B
 P 8300 4750
-F 0 "#PWR013" H 8300 4500 50  0001 C CNN
+F 0 "#PWR012" H 8300 4500 50  0001 C CNN
 F 1 "GND" H 8300 4600 50  0000 C CNN
 F 2 "" H 8300 4750 50  0000 C CNN
@@
 	8400 4750 8300 4750
 $Comp
-L +3.3V #PWR014
+L +3.3V #PWR013
 U 1 1 572D98DD
 P 8100 5000
-F 0 "#PWR014" H 8100 4850 50  0001 C CNN
+F 0 "#PWR013" H 8100 4850 50  0001 C CNN
 F 1 "+3.3V" H 8100 5140 50  0000 C CNN
 F 2 "" H 8100 5000 50  0000 C CNN
@@
 Wire Wire Line
 	8100 5000 8400 5000
-Wire Wire Line
-	7100 4750 7400 4750
-Entry Wire Line
-	7400 4750 7500 4850
-Text Label 7150 4750 0    60   ~ 0
-IR_IN
 Text Label 7650 5100 0    60   ~ 0
 IR_IN
@@
 Connection ~ 5450 6350
 $Comp
-L GND #PWR015
+L GND #PWR014
 U 1 1 572E5080
 P 5450 6400
-F 0 "#PWR015" H 5450 6150 50  0001 C CNN
+F 0 "#PWR014" H 5450 6150 50  0001 C CNN
 F 1 "GND" H 5450 6250 50  0000 C CNN
 F 2 "" H 5450 6400 50  0000 C CNN
@@
 VBR
 $Comp
-L GND #PWR016
+L GND #PWR015
 U 1 1 572EF82E
 P 8500 1650
-F 0 "#PWR016" H 8500 1400 50  0001 C CNN
+F 0 "#PWR015" H 8500 1400 50  0001 C CNN
 F 1 "GND" H 8500 1500 50  0000 C CNN
 F 2 "" H 8500 1650 50  0000 C CNN
@@
 	0    1    1    0
 $EndComp
+Wire Wire Line
+	7100 2450 7400 2450
+Text Label 7400 2450 2    60   ~ 0
+IR_IN
+$Comp
+L CONN_02X04 J1
+U 1 1 595AE1AE
+P 9550 1550
+F 0 "J1" H 9550 1800 50  0000 C CNN
+F 1 "CONN_02X04" H 9550 1300 50  0000 C CNN
+F 2 "Pin_Headers:Pin_Header_Straight_2x04_Pitch2.54mm" H 9550 350 50  0001 C CNN
+F 3 "" H 9550 350 50  0001 C CNN
+	1    9550 1550
+	0    1    1    0
+$EndComp
+Wire Wire Line
+	9400 1300 9400 1000
+Wire Wire Line
+	9500 1200 9500 1300
+Wire Wire Line
+	9600 1200 9600 1300
+Wire Wire Line
+	9700 1300 9700 1000
+Wire Wire Line
+	9400 1800 9400 1800
+Wire Wire Line
+	9500 1800 9500 1850
+Wire Wire Line
+	9600 1800 9600 1800
+Wire Wire Line
+	9600 1800 9600 1950
+Wire Wire Line
+	9700 1800 9700 1950
+$Comp
+L +3.3V #PWR016
+U 1 1 595AF7EE
+P 9400 1000
+F 0 "#PWR016" H 9400 850 50  0001 C CNN
+F 1 "+3.3V" H 9400 1140 50  0000 C CNN
+F 2 "" H 9400 1000 50  0001 C CNN
+F 3 "" H 9400 1000 50  0001 C CNN
+	1    9400 1000
+	1    0    0    -1
+$EndComp
+$Comp
+L R_Small R9
+U 1 1 595AF914
+P 9500 1100
+F 0 "R9" H 9530 1120 50  0001 L CNN
+F 1 "RST" H 9530 1060 50  0001 L CNN
+F 2 "Resistors_ThroughHole:R_Axial_DIN0204_L3.6mm_D1.6mm_P2.54mm_Vertical" H 9500 1100 50  0001 C CNN
+F 3 "" H 9500 1100 50  0001 C CNN
+	1    9500 1100
+	1    0    0    -1
+$EndComp
+Wire Wire Line
+	9400 1000 9600 1000
+Text Label 9700 1000 3    60   ~ 0
+SDA
+Text Notes 9700 950  1    60   ~ 0
+GPIO 01
+$Comp
+L GND #PWR017
+U 1 1 595B47CF
+P 9700 1950
+F 0 "#PWR017" H 9700 1700 50  0001 C CNN
+F 1 "GND" H 9700 1800 50  0000 C CNN
+F 2 "" H 9700 1950 50  0001 C CNN
+F 3 "" H 9700 1950 50  0001 C CNN
+	1    9700 1950
+	1    0    0    -1
+$EndComp
+Text Label 9600 1950 1    60   ~ 0
+SCL
+Text Notes 9600 2200 3    60   ~ 0
+GPIO 02
+$Comp
+L R_Small R11
+U 1 1 595B5E24
+P 9600 1100
+F 0 "R11" H 9630 1120 50  0001 L CNN
+F 1 "RST" H 9630 1060 50  0001 L CNN
+F 2 "Resistors_ThroughHole:R_Axial_DIN0204_L3.6mm_D1.6mm_P2.54mm_Vertical" H 9600 1100 50  0001 C CNN
+F 3 "" H 9600 1100 50  0001 C CNN
+	1    9600 1100
+	1    0    0    -1
+$EndComp
+Connection ~ 9500 1000
+$Comp
+L R_Small R10
+U 1 1 595B61BF
+P 9500 1950
+F 0 "R10" H 9530 1970 50  0001 L CNN
+F 1 "RST" H 9530 1910 50  0001 L CNN
+F 2 "Resistors_ThroughHole:R_Axial_DIN0204_L3.6mm_D1.6mm_P2.54mm_Vertical" H 9500 1950 50  0001 C CNN
+F 3 "" H 9500 1950 50  0001 C CNN
+	1    9500 1950
+	1    0    0    -1
+$EndComp
+Text Label 9400 1800 3    60   ~ 0
+HIT_REC
+Text Notes 9400 2200 3    60   ~ 0
+GPIO 03
+$Comp
+L +3.3V #PWR018
+U 1 1 595BB768
+P 9500 2050
+F 0 "#PWR018" H 9500 1900 50  0001 C CNN
+F 1 "+3.3V" H 9500 2190 50  0000 C CNN
+F 2 "" H 9500 2050 50  0001 C CNN
+F 3 "" H 9500 2050 50  0001 C CNN
+	1    9500 2050
+	-1   0    0    1
+$EndComp
+$Comp
+L C C3
+U 1 1 595C0FD8
+P 4900 3300
+F 0 "C3" H 4925 3400 50  0000 L CNN
+F 1 "22uF" H 4925 3200 50  0000 L CNN
+F 2 "Capacitors_ThroughHole:CP_Radial_D5.0mm_P2.50mm" H 4938 3150 50  0001 C CNN
+F 3 "" H 4900 3300 50  0001 C CNN
+	1    4900 3300
+	1    0    0    -1
+$EndComp
+Wire Wire Line
+	4900 3050 4900 3150
+Wire Wire Line
+	4900 3450 4900 3550
+$Comp
+L GND #PWR019
+U 1 1 595C115B
+P 4900 3550
+F 0 "#PWR019" H 4900 3300 50  0001 C CNN
+F 1 "GND" H 4900 3400 50  0000 C CNN
+F 2 "" H 4900 3550 50  0001 C CNN
+F 3 "" H 4900 3550 50  0001 C CNN
+	1    4900 3550
+	1    0    0    -1
+$EndComp
+$Comp
+L C C?
+U 1 1 595C4950
+P 2200 2000
+F 0 "C?" H 2225 2100 50  0000 L CNN
+F 1 "22uF" H 2225 1900 50  0000 L CNN
+F 2 "" H 2238 1850 50  0001 C CNN
+F 3 "" H 2200 2000 50  0001 C CNN
+	1    2200 2000
+	0    -1   -1   0
+$EndComp
+Wire Wire Line
+	2350 2000 2350 2050
+Wire Wire Line
+	2350 2050 2400 2100
+Wire Wire Line
+	2050 2000 2050 2150
+Wire Wire Line
+	2050 2150 2000 2200
+Connection ~ 2000 2200
+Wire Wire Line
+	1500 1700 1200 1700
 $EndSCHEMATC
