File: Electronics/MainBoard/MainBoard.sch (KiCad schematic (older format))
At the start: 24 parts, among them CN3 RCable_Con_VEST, J1 CONN_02X04, M1 Vibr_Motor, Q1 Q_PNP_CBE, SW1 SW_PUSH, SW2 SPST, U1 ATMEGA168PA-AU

Commit message: Preparing for major PCB changes!
Parts:
- removed CN3: RCable_Con_VEST, Pin_Headers:Pin_Header_Angled_2x05, symbol RCable_Con_VEST
- removed Q1: Q_PNP_CBE, TO_SOT_Packages_THT:TO-92_Inline_Wide, symbol Q_PNP_CBE
- removed R3, R4, R5: 220Ω, Resistors_SMD:R_0603_HandSoldering, symbol R_Small
- added D4, D5: LED_RGBA, LEDs:LED_Cree-PLCC4_3.2x2.8mm_CCW, symbol LED_RGBA
- added J2: DB9_Female, Connectors_DSub:DSUB-9_Female_Horizontal_Pitch2.77x2.84mm_EdgePinOffset4.94mm_Housed_MountingHolesOffset7.48mm, symbol DB9_Female
- added Q1, Q2, Q3, Q4: 2N 2222A, TO_SOT_Packages_SMD:SOT-23_Handsoldering, symbol Q_NPN_BEC
- added RN1, RN3: 220Ω, Resistors_SMD:R_Array_Convex_4x1206, symbol R_Pack04
- added RN2: 100Ω, Resistors_SMD:R_Array_Convex_4x1206, symbol R_Pack04
- C4: value CP -> 100uF; footprint Capacitors_ThroughHole:CP_Radial_D4.0mm_P2.00mm -> Capacitors_SMD:CP_Elec_6.3x5.7; URL (none) -> https://www.reichelt.de/Elkos-SMD-Low-ESR-105-C/SMD-ELKO-10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
Connections:
- net +3V3: now also D4.4 (A), D5.4 (A), J2.6
- net B_MZL: now also RN1.4 (R4.1)
- net GND: now also J2.1, Q1.2 (E), Q2.2 (E), Q3.2 (E), Q4.2 (E)
- net G_MZL: now also RN1.3 (R3.1)
- net IR_IN: now also J2.2
- net IR_LED: now also RN1.1 (R1.1); no longer R1.1
- net MISO: now also RN3.2 (R2.1)
- net MOSI: now also RN3.1 (R1.1)
- net R_MZL: now also RN1.2 (R2.1)
- net SCK: now also RN3.3 (R3.1)
- net SCL: now also J2.9
- net SDA: now also J2.4
- net at D1.1 (K): now also Q1.3 (C)
- net at D2.1 (RED_ANODE): now also RN1.5 (R4.2)
- net at D2.3 (BLUE_ANODE): now also RN1.7 (R2.2)
- net at D2.4 (GREEN_ANODE): now also RN1.6 (R3.2)
- net at R1.2: now also Q1.1 (B)
- new net: R1.1, RN1.8 (R1.2)
- new net: D4.1 (RK), D5.1 (RK), RN2.8 (R1.2)
- new net: D4.2 (GK), D5.2 (GK), RN2.7 (R2.2)
- new net: D4.3 (BK), D5.3 (BK), RN2.6 (R3.2)
- new net: Q3.1 (B), RN3.7 (R2.2)
- new net: Q2.1 (B), RN3.6 (R3.2)
- new net: Q4.1 (B), RN3.8 (R1.2)
- new net B_PWR: J2.8, Q2.3 (C), RN2.3 (R3.1)
- new net G_PWR: J2.3, Q3.3 (C), RN2.2 (R2.1)
- new net R_PWR: J2.7, Q4.3 (C), RN2.1 (R1.1)
Other:
- moved on the sheet: C4, D1, D2, R1

Commit message: More SMD additions
Parts:
- removed D3: D, Discret:R1, symbol D
- removed R1: 220Ω, Resistors_SMD:R_0603_HandSoldering, symbol R
- BT1: footprint Main-Cache:SolderWirePad_2x_0-8mmDrill -> Connectors_JST:JST_PH_S2B-PH-K_02x2.00mm_Angled
- D1: footprint LEDs:LED-3MM -> LEDs:LED_D3.0mm_Horizontal_O1.27mm_Z10.0mm
- D2: footprint LEDs:LED-RGB-5MM_Common_Cathode -> LEDs:LED_D5.0mm-4
- SP1: footprint Buzzers_Beepers:BUZZER -> Buzzers_Beepers:Buzzer_15x7.5RM7.6
- SPI1: footprint Pin_Headers:Pin_Header_Angled_2x03 -> Pin_Headers:Pin_Header_Straight_2x03_Pitch2.54mm
- SW2: footprint Buttons_Switches_ThroughHole:SW_DIP_x1_Slide -> Pin_Headers:Pin_Header_Straight_1x03_Pitch2.54mm
Connections:
- net at BT1.1: now also SW2.1
- net at RN1.8 (R1.2): now also Q1.1 (B)
Other:
- moved on the sheet: SW2
Changed lines of the file:
@@
 F 0 "BT1" H 10350 5750 50  0000 L CNN
 F 1 "Battery" H 10350 5650 50  0000 L CNN
-F 2 "Main-Cache:SolderWirePad_2x_0-8mmDrill" V 10250 5740 50  0001 C CNN
+F 2 "Connectors_JST:JST_PH_S2B-PH-K_02x2.00mm_Angled" V 10250 5740 50  0001 C CNN
 F 3 "" V 10250 5740 50  0000 C CNN
 	1    10250 5700
@@
 F 0 "SPI1" H 8150 1750 50  0000 C CNN
 F 1 "CONN_02X03" H 8150 1350 50  0000 C CNN
-F 2 "Pin_Headers:Pin_Header_Angled_2x03" H 8150 350 50  0001 C CNN
+F 2 "Pin_Headers:Pin_Header_Straight_2x03_Pitch2.54mm" H 8150 350 50  0001 C CNN
 F 3 "" H 8150 350 50  0000 C CNN
 	1    8150 1550
@@
 F 0 "D1" H 2400 2675 50  0000 C CNN
 F 1 "LED" H 2400 2475 50  0000 C CNN
-F 2 "LEDs:LED-3MM" H 2400 2575 50  0001 C CNN
+F 2 "LEDs:LED_D3.0mm_Horizontal_O1.27mm_Z10.0mm" H 2400 2575 50  0001 C CNN
 F 3 "" H 2400 2575 50  0000 C CNN
 	1    2400 2575
@@
 L +3.3V #PWR05
 U 1 1 572B6F24
-P 10250 4250
-F 0 "#PWR05" H 10250 4100 50  0001 C CNN
-F 1 "+3.3V" H 10250 4390 50  0000 C CNN
-F 2 "" H 10250 4250 50  0000 C CNN
-F 3 "" H 10250 4250 50  0000 C CNN
-	1    10250 4250
+P 10250 4550
+F 0 "#PWR05" H 10250 4400 50  0001 C CNN
+F 1 "+3.3V" H 10250 4690 50  0000 C CNN
+F 2 "" H 10250 4550 50  0000 C CNN
+F 3 "" H 10250 4550 50  0000 C CNN
+	1    10250 4550
 	1    0    0    -1
 $EndComp
@@
 F 0 "D2" H 2100 3825 50  0000 C CNN
 F 1 "LED_RCBG" H 2100 3125 50  0000 C CNN
-F 2 "LEDs:LED-RGB-5MM_Common_Cathode" H 2100 3425 50  0001 C CNN
+F 2 "LEDs:LED_D5.0mm-4" H 2100 3425 50  0001 C CNN
 F 3 "" H 2100 3425 50  0000 C CNN
 	1    2100 3475
@@
 L SPST SW2
 U 1 1 572DFDFF
-P 10250 4750
-F 0 "SW2" H 10250 4850 50  0000 C CNN
-F 1 "SPST" H 10250 4650 50  0000 C CNN
-F 2 "Buttons_Switches_ThroughHole:SW_DIP_x1_Slide" H 10250 4750 50  0001 C CNN
-F 3 "" H 10250 4750 50  0000 C CNN
-	1    10250 4750
+P 10250 5050
+F 0 "SW2" H 10250 5150 50  0000 C CNN
+F 1 "SPST" H 10250 4950 50  0000 C CNN
+F 2 "Pin_Headers:Pin_Header_Straight_1x03_Pitch2.54mm" H 10250 5050 50  0001 C CNN
+F 3 "" H 10250 5050 50  0000 C CNN
+	1    10250 5050
 	0    -1   -1   0
 $EndComp
@@
 F 0 "SP1" H 5700 5550 50  0000 C CNN
 F 1 "SPEAKER" H 5700 5050 50  0000 C CNN
-F 2 "Buzzers_Beepers:BUZZER" H 5800 5300 50  0001 C CNN
+F 2 "Buzzers_Beepers:Buzzer_15x7.5RM7.6" H 5800 5300 50  0001 C CNN
 F 3 "" H 5800 5300 50  0000 C CNN
 	1    5800 5300
@@
 	1    8500 1650
 	1    0    0    -1
-$EndComp
-$Comp
-L D D3
-U 1 1 572DFB0F
-P 10250 5400
-F 0 "D3" H 10250 5500 50  0000 C CNN
-F 1 "D" H 10250 5300 50  0000 C CNN
-F 2 "Discret:R1" H 10250 5400 50  0001 C CNN
-F 3 "" H 10250 5400 50  0000 C CNN
-	1    10250 5400
-	0    1    1    0
 $EndComp
 Text Label 7400 2450 2    60   ~ 0
@@
 	1    2400 3775
 	1    0    0    -1
-$EndComp
-$Comp
-L R R1
-U 1 1 59700C12
-P 1950 2975
-F 0 "R1" V 2030 2975 50  0000 C CNN
-F 1 "220Ω" V 1950 2975 50  0000 C CNN
-F 2 "Resistors_SMD:R_0603_HandSoldering" V 1880 2975 50  0001 C CNN
-F 3 "" H 1950 2975 50  0001 C CNN
-	1    1950 2975
-	0    -1   -1   0
 $EndComp
 Text Label 1150 3225 2    60   ~ 0
@@
 $EndComp
 Wire Wire Line
-	7900 3200 8300 3200
-Wire Wire Line
-	7900 3000 8300 3000
+	7900 3200 8100 3200
+Wire Wire Line
+	8100 3200 8300 3200
+Wire Wire Line
+	7900 3000 8100 3000
+Wire Wire Line
+	8100 3000 8300 3000
 Wire Wire Line
 	8500 3000 8500 3200
@@
 Connection ~ 8100 3200
 Wire Wire Line
-	5200 4550 5200 4800
+	5200 4550 5200 4650
+Wire Wire Line
+	5200 4650 5200 4750
+Wire Wire Line
+	5200 4750 5200 4800
 Connection ~ 5200 4750
 Wire Wire Line
-	5200 2450 5200 2750
-Wire Bus Line
-	7500 1850 7500 5900
+	5200 2450 5200 2550
+Wire Wire Line
+	5200 2550 5200 2750
+Wire Bus Line
+	7500 1850 7500 2350
+Wire Bus Line
+	7500 2350 7500 2850
+Wire Bus Line
+	7500 2850 7500 2950
+Wire Bus Line
+	7500 2950 7500 3050
+Wire Bus Line
+	7500 3050 7500 3800
+Wire Bus Line
+	7500 3800 7500 3900
+Wire Bus Line
+	7500 3900 7500 4000
+Wire Bus Line
+	7500 4000 7500 4150
+Wire Bus Line
+	7500 4150 7500 4250
+Wire Bus Line
+	7500 4250 7500 4450
+Wire Bus Line
+	7500 4450 7500 4550
+Wire Bus Line
+	7500 4550 7500 4650
+Wire Bus Line
+	7500 4650 7500 4750
+Wire Bus Line
+	7500 4750 7500 5200
+Wire Bus Line
+	7500 5200 7500 5600
+Wire Bus Line
+	7500 5600 7500 5700
+Wire Bus Line
+	7500 5700 7500 5800
+Wire Bus Line
+	7500 5800 7500 5900
 Wire Wire Line
 	7900 1450 7700 1450
@@
 	8400 1450 8500 1450
 Wire Bus Line
-	7600 1550 7600 1850
+	7600 1550 7600 1650
+Wire Bus Line
+	7600 1650 7600 1750
+Wire Bus Line
+	7600 1750 7600 1850
 Wire Bus Line
 	8600 1850 7500 1850
@@
 	7900 3050 7900 3000
 Wire Wire Line
-	2400 3175 2400 3775
+	2400 3175 2400 3225
+Wire Wire Line
+	2400 3225 2400 3475
+Wire Wire Line
+	2400 3475 2400 3775
 Connection ~ 2400 3475
 Wire Wire Line
@@
 	5700 5600 5450 5600
 Wire Wire Line
-	5450 5600 5450 6400
+	5450 5600 5450 5900
+Wire Wire Line
+	5450 5900 5450 6350
+Wire Wire Line
+	5450 6350 5450 6400
 Wire Wire Line
 	5450 5900 5500 5900
@@
 	9700 1800 9700 1950
 Wire Wire Line
-	9400 1000 9600 1000
+	9400 1000 9500 1000
+Wire Wire Line
+	9500 1000 9600 1000
 Connection ~ 9500 1000
 Wire Wire Line
@@
 	7100 3600 7400 3600
 Wire Wire Line
-	2400 2125 2400 2375
+	2400 2125 2400 2175
+Wire Wire Line
+	2400 2175 2400 2325
+Wire Wire Line
+	2400 2325 2400 2375
 Connection ~ 2400 2325
 Connection ~ 2400 3225
@@
 	4500 2550 4600 2550
 Wire Wire Line
-	4600 2450 4600 3400
+	4600 2450 4600 2550
+Wire Wire Line
+	4600 2550 4600 3400
 Wire Wire Line
 	4600 3400 4500 3400
@@
 Connection ~ 4600 2550
 Wire Wire Line
-	3725 2350 4100 2350
+	3725 2350 4000 2350
+Wire Wire Line
+	4000 2350 4100 2350
 Wire Wire Line
 	4100 2550 3950 2550
@@
 	3725 2450 3950 2450
 Wire Wire Line
-	3950 2450 3950 3400
+	3950 2450 3950 2550
+Wire Wire Line
+	3950 2550 3950 3400
 Wire Wire Line
 	3725 2550 3900 2550
 Wire Wire Line
-	3900 2550 3900 3600
+	3900 2550 3900 2750
+Wire Wire Line
+	3900 2750 3900 3600
 Connection ~ 3900 2750
 Connection ~ 3950 2550
@@
 	1650 3125 1650 2975
 Wire Wire Line
-	1650 2975 1800 2975
+	1650 2975 2100 2975
 Wire Wire Line
 	1650 3225 1800 3225

Commit message: Final small changes
Parts:
- added Q5: 2N 2222A, TO_SOT_Packages_SMD:SOT-23_Handsoldering, symbol Q_NPN_BEC
- added R1: 470Ω, Resistors_SMD:R_0603_HandSoldering, symbol R_Small
- C4: value 100uF -> 22uF; footprint Capacitors_SMD:CP_Elec_6.3x5.7 -> Capacitors_SMD:CP_Elec_5x5.3; URL https://www.reichelt.de/Elkos-SMD-Low-ESR-105-C/SMD-ELKO-10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 -> https://www.reichelt.de/Elkos-SMD-Low-ESR-105-C/SMD-ELKO-22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
Connections:
- net +3V3: now also M1.2 (Vcc); no longer C4.1
- net GND: now also Q5.2 (E); no longer M1.1 (GND)
- net VBR: now also R1.2; no longer M1.2 (Vcc)
- net at BT1.1, SW2.1: now also C4.1
- net V_VBR: now reaches U1.11 ((PCINT23/AIN1)PD7)
- net V_VBR: now also J2.5
- new net: M1.1 (GND), Q5.3 (C)
- new net: Q5.1 (B), R1.1
Other:
- moved on the sheet: BT1, C4, M1

Commit message: Finalized schematics and Gerbers - for now
Parts:
- BT1: footprint Connectors_JST:JST_PH_S2B-PH-K_02x2.00mm_Angled -> Connectors_JST:JST_PH_B2B-PH-K_02x2.00mm_Straight; URL (none) -> https://www.reichelt.de/JST-Vielfachsteckverbinder/JST-PH2P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
- M1, SW1: footprint Main-Cache:SolderWirePad_2x_0-8mmDrill -> Pin_Headers:Pin_Header_Straight_1x02_Pitch2.54mm
- QRZ1: value Crystal_Small -> 4MHz
- RN1, RN3: footprint Resistors_SMD:R_Array_Convex_4x1206 -> Resistors_SMD:R_Array_Convex_4x0603
- RN2: value 100Ω -> 220Ω; footprint Resistors_SMD:R_Array_Convex_4x1206 -> Resistors_SMD:R_Array_Convex_4x0603
Changed lines of the file:
@@
 P 8100 3100
 F 0 "QRZ1" H 8100 3200 50  0000 C CNN
-F 1 "Crystal_Small" H 8100 3000 50  0000 C CNN
+F 1 "4MHz" H 8100 3000 50  0000 C CNN
 F 2 "Crystals:Crystal_HC49-U_Vertical" H 8100 3100 50  0001 C CNN
 F 3 "" H 8100 3100 50  0000 C CNN
@@
 F 0 "BT1" H 10350 5800 50  0000 L CNN
 F 1 "Battery" H 10350 5700 50  0000 L CNN
-F 2 "Connectors_JST:JST_PH_S2B-PH-K_02x2.00mm_Angled" V 10250 5790 50  0001 C CNN
+F 2 "Connectors_JST:JST_PH_B2B-PH-K_02x2.00mm_Straight" V 10250 5790 50  0001 C CNN
 F 3 "" V 10250 5790 50  0000 C CNN
+F 4 "https://www.reichelt.de/JST-Vielfachsteckverbinder/JST-PH2P-ST/3/index.html?ACTION=3&LA=2&ARTICLE=185049&GROUPID=7980&artnr=JST+PH2P+ST&trstct=pol_7" H 10250 5750 60  0001 C CNN "URL"
 	1    10250 5750
 	1    0    0    -1
@@
 F 1 "1MΩ" H 7980 2110 50  0000 L CNN
 F 2 "Resistors_SMD:R_0603_HandSoldering" H 7950 2150 50  0001 C CNN
-F 3 "" H 7950 2150 50  0000 C CNN
+F 3 "https://www.reichelt.de/SMD-0603-von-1-bis-910-kOhm/RND-0603-1-100K/3/index.html?ACTION=3&LA=2&ARTICLE=183102&GROUPID=7968&artnr=RND+0603+1+100K&trstct=pol_1;SID=94WOY5-qwQATcAAG79Goo0acb105dd429f907499a137e0497339a" H 7950 2150 50  0001 C CNN
 	1    7950 2150
 	1    0    0    -1
@@
 F 0 "SW1" H 5950 6010 50  0000 C CNN
 F 1 "SW_PUSH" H 5800 5820 50  0000 C CNN
-F 2 "Main-Cache:SolderWirePad_2x_0-8mmDrill" H 5800 5900 50  0001 C CNN
+F 2 "Pin_Headers:Pin_Header_Straight_1x02_Pitch2.54mm" H 5800 5900 50  0001 C CNN
 F 3 "" H 5800 5900 50  0000 C CNN
 	1    5800 5900
@@
 F 0 "M1" H 6350 6575 60  0000 C CNN
 F 1 "Vibr_Motor" H 6150 6675 60  0000 C CNN
-F 2 "Main-Cache:SolderWirePad_2x_0-8mmDrill" H 6000 6625 60  0001 C CNN
+F 2 "Pin_Headers:Pin_Header_Straight_1x02_Pitch2.54mm" H 6000 6625 60  0001 C CNN
 F 3 "" H 6000 6625 60  0000 C CNN
 	1    6100 6625
@@
 F 1 "RST" H 9530 1060 50  0001 L CNN
 F 2 "Resistors_SMD:R_0603_HandSoldering" H 9500 1100 50  0001 C CNN
-F 3 "" H 9500 1100 50  0001 C CNN
+F 3 "https://www.reichelt.de/SMD-0603-von-1-bis-910-kOhm/RND-0603-1-100K/3/index.html?ACTION=3&LA=2&ARTICLE=183102&GROUPID=7968&artnr=RND+0603+1+100K&trstct=pol_1;SID=94WOY5-qwQATcAAG79Goo0acb105dd429f907499a137e0497339a" H 9500 1100 50  0001 C CNN
 	1    9500 1100
 	1    0    0    -1
@@
 F 1 "RST" H 9630 1060 50  0001 L CNN
 F 2 "Resistors_SMD:R_0603_HandSoldering" H 9600 1100 50  0001 C CNN
-F 3 "" H 9600 1100 50  0001 C CNN
+F 3 "https://www.reichelt.de/SMD-0603-von-1-bis-910-kOhm/RND-0603-1-100K/3/index.html?ACTION=3&LA=2&ARTICLE=183102&GROUPID=7968&artnr=RND+0603+1+100K&trstct=pol_1;SID=94WOY5-qwQATcAAG79Goo0acb105dd429f907499a137e0497339a" H 9600 1100 50  0001 C CNN
 	1    9600 1100
 	1    0    0    -1
@@
 P 3525 2550
 F 0 "RN2" V 3225 2550 50  0000 C CNN
-F 1 "100Ω" V 3725 2550 50  0000 C CNN
-F 2 "Resistors_SMD:R_Array_Convex_4x1206" V 3800 2550 50  0001 C CNN
-F 3 "" H 3525 2550 50  0001 C CNN
+F 1 "220Ω" V 3725 2550 50  0000 C CNN
+F 2 "Resistors_SMD:R_Array_Convex_4x0603" V 3800 2550 50  0001 C CNN
+F 3 "https://www.reichelt.de/4-Widerstaende-SMD-1206/BCN16-220/3/index.html?ACTION=3&LA=2&ARTICLE=42464&GROUPID=4495&artnr=BCN16+220&trstct=pol_0" H 3525 2550 50  0001 C CNN
 	1    3525 2550
 	0    1    1    0
@@
 F 0 "RN1" V 1150 3325 50  0000 C CNN
 F 1 "220Ω" V 1650 3325 50  0000 C CNN
-F 2 "Resistors_SMD:R_Array_Convex_4x1206" V 1725 3325 50  0001 C CNN
-F 3 "" H 1450 3325 50  0001 C CNN
+F 2 "Resistors_SMD:R_Array_Convex_4x0603" V 1725 3325 50  0001 C CNN
+F 3 "https://www.reichelt.de/4-Widerstaende-SMD-1206/BCN16-220/3/index.html?ACTION=3&LA=2&ARTICLE=42464&GROUPID=4495&artnr=BCN16+220&trstct=pol_0" H 1450 3325 50  0001 C CNN
 	1    1450 3325
 	0    1    1    0
@@
 F 0 "RN3" V 9000 3250 50  0000 C CNN
 F 1 "220Ω" V 9500 3250 50  0000 C CNN
-F 2 "Resistors_SMD:R_Array_Convex_4x1206" V 9575 3250 50  0001 C CNN
-F 3 "" H 9300 3250 50  0001 C CNN
+F 2 "Resistors_SMD:R_Array_Convex_4x0603" V 9575 3250 50  0001 C CNN
+F 3 "https://www.reichelt.de/4-Widerstaende-SMD-1206/BCN16-220/3/index.html?ACTION=3&LA=2&ARTICLE=42464&GROUPID=4495&artnr=BCN16+220&trstct=pol_0" H 9300 3250 50  0001 C CNN
 	1    9300 3250
 	0    1    1    0

Commit message: Last few tweaks, i.e. fixing ground plane
Parts:
- BT1: symbol Battery-RESCUE-MainBoard -> MainBoard-rescue:Battery-RESCUE-MainBoard
- C1, C2: symbol C_Small -> MainBoard-rescue:C_Small
- C4: symbol CP -> MainBoard-rescue:CP
- D1: symbol LED-RESCUE-MainBoard -> MainBoard-rescue:LED-RESCUE-MainBoard
- D2: symbol LED_RCBG-RESCUE-MainBoard -> MainBoard-rescue:LED_RCBG-RESCUE-MainBoard
- D4, D5: symbol LED_RGBA -> MainBoard-rescue:LED_RGBA
- J1: symbol CONN_02X04 -> MainBoard-rescue:CONN_02X04
- J2: symbol DB9_Female -> MainBoard-rescue:DB9_Female
- M1: symbol Vibr_Motor -> MainBoard-rescue:Vibr_Motor
- Q1, Q2, Q3, Q4, Q5: symbol Q_NPN_BEC -> MainBoard-rescue:Q_NPN_BEC
- QRZ1: symbol Crystal_Small -> MainBoard-rescue:Crystal_Small
- R1, R11, R6, R9: symbol R_Small -> MainBoard-rescue:R_Small
- RN1, RN2, RN3: symbol R_Pack04 -> MainBoard-rescue:R_Pack04
- SP1: symbol SPEAKER -> MainBoard-rescue:SPEAKER
- SPI1: symbol CONN_02X03 -> MainBoard-rescue:CONN_02X03
- SW1: symbol SW_PUSH -> MainBoard-rescue:SW_PUSH
- SW2: symbol SPST -> MainBoard-rescue:SPST
- U1: symbol ATMEGA168PA-AU -> MainBoard-rescue:ATMEGA168PA-AU
