File: Electronics/MainBoard_Rev2/Peripherals.sch (KiCad schematic (older format))
At the start: 18 parts

Commit message: Rev 3.0 is now done!
Parts:
- removed D?: WS2812B, LED_THT:LED_D5.0mm-4_RGB, symbol LED:WS2812B
- added D1: WS2812B_5mm, LED_THT:LED_D5.0mm-4_RGB, symbol TP301:WS2812B_5mm
- added D3, D5: WS2812B, LED_SMD:LED_WS2812B_PLCC4_5.0x5.0mm_P3.2mm, symbol LED:WS2812B
- AMP1: renamed from AMP?; Digi-Key (none) -> 296-1945-1-ND; DigiKey 296-1945-1-ND -> (none); MPN (none) -> TPA301DR
- C31, C38, C39: renamed from C?; footprint (none) -> Capacitor_SMD:C_0603_1608Metric
- D2: renamed from D?; Digi-Key (none) -> 1528-1104-ND
- D30: renamed from D?; Digi-Key (none) -> 475-3581-ND; MPN (none) -> SFH 4346
- D35: renamed from D?; footprint (none) -> Diode_SMD:D_0603_1608Metric
- LS1: renamed from LS?; footprint (none) -> Connector_PinHeader_2.54mm:PinHeader_1x02_P2.54mm_Vertical; Digi-Key (none) -> 102-2502-ND; MPN (none) -> CDM-20008
- R30, R35, R38, R39: renamed from R?; footprint (none) -> Resistor_SMD:R_0603_1608Metric
- TRGR1: renamed from SW?; footprint (none) -> Connector_PinHeader_2.54mm:PinHeader_1x02_P2.54mm_Vertical
- VBR1: renamed from VBR; footprint (none) -> Connector_PinHeader_2.54mm:PinHeader_1x02_P2.54mm_Vertical; Digi-Key (none) -> 1597-1244-ND; MPN (none) -> 316040001
- gave numbers to parts that had none: 3
Connections:
- wire segments 36 -> 42
- no-connect marks 0 -> 2
Other:
- moved on the sheet: C31, C38, C39, D2, D30, D35, D4, Q30, Q35, R30, R35, R38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

Commit message: Began preparing a branch for HackADay users
Parts:
- removed AMP1: TPA301, Package_SO:SOIC-8_3.9x4.9mm_P1.27mm, symbol TP301:TPA301
- removed C38, C39: 150nF, Capacitor_SMD:C_0603_1608Metric, symbol Device:C_Small
- removed LS1: Speaker, Connector_PinHeader_2.54mm:PinHeader_1x02_P2.54mm_Vertical, symbol Device:Speaker
- removed R38: 10k, Resistor_SMD:R_0603_1608Metric, symbol Device:R_Small
- removed R39: 20k-50k, Resistor_SMD:R_0603_1608Metric, symbol Device:R_Small
Connections:
- net labels removed: Audio_In
- wire segments 42 -> 28
Changed lines of the file:
@@
 	4625 3500 4825 3500
-$Comp
-L power:GND #PWR0125
-U 1 1 5C2D7315
-P 9125 2400
-F 0 "#PWR0125" H 9125 2150 50  0001 C CNN
-F 1 "GND" H 9130 2227 50  0000 C CNN
-F 2 "" H 9125 2400 50  0001 C CNN
-F 3 "" H 9125 2400 50  0001 C CNN
-	1    9125 2400
-	1    0    0    -1
-$EndComp
-Wire Wire Line
-	8650 1700 8700 1700
 $Comp
 L Switch:SW_Push TRGR1
@@
 Wire Wire Line
 	9875 5000 9875 4850
-$Comp
-L TP301:TPA301 AMP1
-U 1 1 5C2EF350
-P 9125 2300
-F 0 "AMP1" H 9375 2150 50  0000 C CNN
-F 1 "TPA301" H 9400 2225 50  0000 C CNN
-F 2 "Package_SO:SOIC-8_3.9x4.9mm_P1.27mm" H 9225 2050 50  0001 C CNN
-F 3 "" H 9125 2300 50  0001 C CNN
-F 4 "296-1945-1-ND" H 9125 3236 50  0001 C CNN "Digi-Key"
-F 5 "TPA301DR" H 9125 2300 50  0001 C CNN "MPN"
-	1    9125 2300
-	1    0    0    -1
-$EndComp
-$Comp
-L Device:Speaker LS1
-U 1 1 5C2EF806
-P 9825 1700
-F 0 "LS1" H 9995 1696 50  0000 L CNN
-F 1 "Speaker" H 9995 1605 50  0000 L CNN
-F 2 "Connector_PinHeader_2.54mm:PinHeader_1x02_P2.54mm_Vertical" H 9825 1500 50  0001 C CNN
-F 3 "~" H 9815 1650 50  0001 C CNN
-F 4 "CDM-20008" H 9825 1700 50  0001 C CNN "MPN"
-F 5 "102-2502-ND" H 9825 1700 50  0001 C CNN "Digi-Key"
-	1    9825 1700
-	1    0    0    -1
-$EndComp
-Wire Wire Line
-	9475 1700 9550 1700
-Wire Wire Line
-	9625 1800 9475 1800
-Wire Wire Line
-	8775 1800 8775 1875
-Wire Wire Line
-	8775 1875 8375 1875
-Connection ~ 8775 1875
-Wire Wire Line
-	8775 1875 8775 1900
-$Comp
-L Device:C_Small C39
-U 1 1 5C2F0C41
-P 8375 2025
-F 0 "C39" H 8467 2071 50  0000 L CNN
-F 1 "150nF" H 8467 1980 50  0000 L CNN
-F 2 "Capacitor_SMD:C_0603_1608Metric" H 8375 2025 50  0001 C CNN
-F 3 "~" H 8375 2025 50  0001 C CNN
-	1    8375 2025
-	1    0    0    -1
-$EndComp
-Wire Wire Line
-	8375 1875 8375 1925
-$Comp
-L power:GND #PWR0131
-U 1 1 5C2F395C
-P 8375 2125
-F 0 "#PWR0131" H 8375 1875 50  0001 C CNN
-F 1 "GND" H 8380 1952 50  0000 C CNN
-F 2 "" H 8375 2125 50  0001 C CNN
-F 3 "" H 8375 2125 50  0001 C CNN
-	1    8375 2125
-	1    0    0    -1
-$EndComp
-$Comp
-L power:+BATT #PWR0132
-U 1 1 5C2F3A03
-P 9125 1450
-F 0 "#PWR0132" H 9125 1300 50  0001 C CNN
-F 1 "+BATT" H 9140 1623 50  0000 C CNN
-F 2 "" H 9125 1450 50  0001 C CNN
-F 3 "" H 9125 1450 50  0001 C CNN
-	1    9125 1450
-	1    0    0    -1
-$EndComp
-Wire Wire Line
-	9550 1700 9550 1200
-Connection ~ 9550 1700
-Wire Wire Line
-	9550 1700 9625 1700
-$Comp
-L Device:R_Small R38
-U 1 1 5C2F4850
-P 8550 1700
-F 0 "R38" V 8354 1700 50  0000 C CNN
-F 1 "10k" V 8445 1700 50  0000 C CNN
-F 2 "Resistor_SMD:R_0603_1608Metric" H 8550 1700 50  0001 C CNN
-F 3 "~" H 8550 1700 50  0001 C CNN
-	1    8550 1700
-	0    1    1    0
-$EndComp
-Wire Wire Line
-	8450 1700 8375 1700
-$Comp
-L Device:R_Small R39
-U 1 1 5C2F5F62
-P 8700 1400
-F 0 "R39" H 8641 1354 50  0000 R CNN
-F 1 "20k-50k" H 8641 1445 50  0000 R CNN
-F 2 "Resistor_SMD:R_0603_1608Metric" H 8700 1400 50  0001 C CNN
-F 3 "~" H 8700 1400 50  0001 C CNN
-	1    8700 1400
-	-1   0    0    1
-$EndComp
-Wire Wire Line
-	8700 1200 8700 1300
-Wire Wire Line
-	8700 1200 9550 1200
-Wire Wire Line
-	8700 1500 8700 1700
-Connection ~ 8700 1700
-Wire Wire Line
-	8700 1700 8775 1700
-$Comp
-L Device:C_Small C38
-U 1 1 5C2F7982
-P 8275 1700
-F 0 "C38" V 8046 1700 50  0000 C CNN
-F 1 "150nF" V 8137 1700 50  0000 C CNN
-F 2 "Capacitor_SMD:C_0603_1608Metric" H 8275 1700 50  0001 C CNN
-F 3 "~" H 8275 1700 50  0001 C CNN
-	1    8275 1700
-	0    1    1    0
-$EndComp
-Text HLabel 8175 1700 0    50   Input ~ 0
-Audio_In
 Wire Wire Line
 	2350 3500 2450 3500

Commit message: Began rework to even better hardware
Parts:
- removed D1: WS2812B_5mm, LED_THT:LED_D5.0mm-4_RGB, symbol TP301:WS2812B_5mm
- added C3: 0.1uF, symbol Device:C_Small
- added U2: WS2811, symbol Driver_LED:WS2811
- added U3: LSM6DS3, Package_LGA:LGA-14_3x2.5mm_P0.5mm_LayoutBorder3x4y, symbol Sensor_Motion:LSM6DS3
Connections:
- net labels added: +3.3V, SCL, SDA
- wire segments 28 -> 49
- no-connect marks 2 -> 4
Changed lines of the file:
@@
 Wire Wire Line
 	3800 3500 4000 3500
-Text HLabel 2350 3500 0    50   Input ~ 0
+Text HLabel 1550 4100 0    50   Input ~ 0
 WS2812B_In
-Wire Wire Line
-	3050 3500 3125 3500
 Text HLabel 4825 3500 2    50   Input ~ 0
 WS2812B_Out
@@
 Wire Wire Line
 	9875 5000 9875 4850
-Wire Wire Line
-	2350 3500 2450 3500
 $Comp
 L power:+BATT #PWR0133
@@
 L power:GND #PWR0134
 U 1 1 5C2FED50
-P 2750 3800
-F 0 "#PWR0134" H 2750 3550 50  0001 C CNN
-F 1 "GND" H 2755 3627 50  0000 C CNN
-F 2 "" H 2750 3800 50  0001 C CNN
-F 3 "" H 2750 3800 50  0001 C CNN
-	1    2750 3800
-	1    0    0    -1
-$EndComp
-$Comp
-L TP301:WS2812B_5mm D1
-U 1 1 5C2DE5D0
-P 2750 3500
-F 0 "D1" H 2550 3750 50  0000 L CNN
-F 1 "WS2812B_5mm" H 2800 3225 50  0000 L CNN
-F 2 "LED_THT:LED_D5.0mm-4_RGB" H 2400 3750 50  0001 C CNN
-F 3 "" H 2750 3500 50  0001 C CNN
-F 4 "1568-1213-ND" H 3091 3409 50  0001 L CNN "Digi-Key"
-	1    2750 3500
+P 2150 4550
+F 0 "#PWR0134" H 2150 4300 50  0001 C CNN
+F 1 "GND" H 2155 4377 50  0000 C CNN
+F 2 "" H 2150 4550 50  0001 C CNN
+F 3 "" H 2150 4550 50  0001 C CNN
+	1    2150 4550
 	1    0    0    -1
 $EndComp
@@
 	4000 3500 4025 3500
 NoConn ~ 3800 4575
+$Comp
+L Sensor_Motion:LSM6DS3 U3
+U 1 1 5D2620F3
+P 6800 2250
+F 0 "U3" H 7441 2296 50  0000 L CNN
+F 1 "LSM6DS3" H 7441 2205 50  0000 L CNN
+F 2 "Package_LGA:LGA-14_3x2.5mm_P0.5mm_LayoutBorder3x4y" H 6400 1550 50  0001 L CNN
+F 3 "www.st.com/resource/en/datasheet/lsm6ds3.pdf" H 6900 1600 50  0001 C CNN
+	1    6800 2250
+	1    0    0    -1
+$EndComp
+Wire Wire Line
+	6200 2150 6200 2050
+Wire Wire Line
+	6200 2050 6200 1950
+Connection ~ 6200 2050
+Wire Wire Line
+	6200 1950 6200 1650
+Wire Wire Line
+	6200 1650 6425 1650
+Connection ~ 6200 1950
+Wire Wire Line
+	6800 1650 6900 1650
+Connection ~ 6800 1650
+$Comp
+L Device:C_Small C3
+U 1 1 5D263C3E
+P 5750 1775
+F 0 "C3" H 5658 1729 50  0000 R CNN
+F 1 "0.1uF" H 5658 1820 50  0000 R CNN
+F 2 "" H 5750 1775 50  0001 C CNN
+F 3 "~" H 5750 1775 50  0001 C CNN
+	1    5750 1775
+	-1   0    0    1
+$EndComp
+Wire Wire Line
+	5750 1675 5750 1650
+Wire Wire Line
+	5750 1650 6200 1650
+Connection ~ 6200 1650
+$Comp
+L power:GND #PWR0132
+U 1 1 5D264301
+P 5750 1925
+F 0 "#PWR0132" H 5750 1675 50  0001 C CNN
+F 1 "GND" H 5755 1752 50  0000 C CNN
+F 2 "" H 5750 1925 50  0001 C CNN
+F 3 "" H 5750 1925 50  0001 C CNN
+	1    5750 1925
+	1    0    0    -1
+$EndComp
+Wire Wire Line
+	5750 1875 5750 1925
+$Comp
+L power:+3.3V #PWR0143
+U 1 1 5D264984
+P 6425 1650
+F 0 "#PWR0143" H 6425 1500 50  0001 C CNN
+F 1 "+3.3V" H 6440 1823 50  0000 C CNN
+F 2 "" H 6425 1650 50  0001 C CNN
+F 3 "" H 6425 1650 50  0001 C CNN
+	1    6425 1650
+	1    0    0    -1
+$EndComp
+Connection ~ 6425 1650
+Wire Wire Line
+	6425 1650 6800 1650
+Wire Wire Line
+	6200 2150 6050 2150
+Wire Wire Line
+	6050 2150 6050 2550
+Wire Wire Line
+	6050 2550 6200 2550
+Connection ~ 6200 2150
+$Comp
+L power:GND #PWR0144
+U 1 1 5D265D9B
+P 6850 2975
+F 0 "#PWR0144" H 6850 2725 50  0001 C CNN
+F 1 "GND" H 6855 2802 50  0000 C CNN
+F 2 "" H 6850 2975 50  0001 C CNN
+F 3 "" H 6850 2975 50  0001 C CNN
+	1    6850 2975
+	1    0    0    -1
+$EndComp
+Wire Wire Line
+	6800 2850 6850 2850
+Wire Wire Line
+	6850 2850 6850 2975
+Connection ~ 6850 2850
+Wire Wire Line
+	6850 2850 6900 2850
+NoConn ~ 7400 1950
+NoConn ~ 7400 2050
+Text GLabel 5800 2350 0    50   Input ~ 0
+SDA
+Text GLabel 5800 2450 0    50   Input ~ 0
+SCL
+Wire Wire Line
+	5800 2350 6200 2350
+Wire Wire Line
+	6200 2450 5800 2450
+$Comp
+L Driver_LED:WS2811 U2
+U 1 1 5D266A84
+P 2150 4200
+F 0 "U2" H 1900 4650 50  0000 C CNN
+F 1 "WS2811" H 1900 4550 50  0000 C CNN
+F 2 "" H 1850 4350 50  0001 C CNN
+F 3 "https://cdn-shop.adafruit.com/datasheets/WS2811.pdf" H 1950 4450 50  0001 C CNN
+	1    2150 4200
+	1    0    0    -1
+$EndComp
+Wire Wire Line
+	1550 4100 1750 4100
+Wire Wire Line
+	1750 4200 1625 4200
+Wire Wire Line
+	1625 4200 1625 3500
+Wire Wire Line
+	1625 3500 3125 3500
+Wire Wire Line
+	2150 4500 2150 4550
+$Comp
+L power:+BATT #PWR0145
+U 1 1 5D26BA5D
+P 2150 3825
+F 0 "#PWR0145" H 2150 3675 50  0001 C CNN
+F 1 "+BATT" H 2165 3998 50  0000 C CNN
+F 2 "" H 2150 3825 50  0001 C CNN
+F 3 "" H 2150 3825 50  0001 C CNN
+	1    2150 3825
+	1    0    0    -1
+$EndComp
+Wire Wire Line
+	2150 3825 2150 3900
 $EndSCHEMATC

Commit message: Fixed footprint assignment
Parts:
- C3: footprint (none) -> Capacitor_SMD:C_0805_2012Metric
- U2: footprint (none) -> Package_SO:SSOP-8_3.95x5.21x3.27mm_P1.27mm
Connections:
- no-connect marks 4 -> 5
Changed lines of the file:
@@
 F 0 "C3" H 5658 1729 50  0000 R CNN
 F 1 "0.1uF" H 5658 1820 50  0000 R CNN
-F 2 "" H 5750 1775 50  0001 C CNN
+F 2 "Capacitor_SMD:C_0805_2012Metric" H 5750 1775 50  0001 C CNN
 F 3 "~" H 5750 1775 50  0001 C CNN
 	1    5750 1775
@@
 F 0 "U2" H 1900 4650 50  0000 C CNN
 F 1 "WS2811" H 1900 4550 50  0000 C CNN
-F 2 "" H 1850 4350 50  0001 C CNN
+F 2 "Package_SO:SSOP-8_3.95x5.21x3.27mm_P1.27mm" H 1850 4350 50  0001 C CNN
 F 3 "https://cdn-shop.adafruit.com/datasheets/WS2811.pdf" H 1950 4450 50  0001 C CNN
 	1    2150 4200
@@
 Wire Wire Line
 	2150 3825 2150 3900
+NoConn ~ 1750 4300
 $EndSCHEMATC

Commit message: Temporary polishing of PCB
Parts:
- removed U2: WS2811, Package_SO:SSOP-8_3.95x5.21x3.27mm_P1.27mm, symbol Driver_LED:WS2811
- added D1: COM-12999, digikey-footprints:LED_RGB_WP154A4SUREQBFZGC, symbol dk_Addressable-Specialty:COM-12999
- C31: footprint Capacitor_SMD:C_0603_1608Metric -> Capacitor_SMD:C_0805_2012Metric
- R30, R35: footprint Resistor_SMD:R_0603_1608Metric -> Resistor_SMD:R_0805_2012Metric
Connections:
- wire segments 49 -> 45
- no-connect marks 5 -> 4
Changed lines of the file:
@@
 Wire Wire Line
 	3800 3500 4000 3500
-Text HLabel 1550 4100 0    50   Input ~ 0
+Text HLabel 1875 3500 0    50   Input ~ 0
 WS2812B_In
 Text HLabel 4825 3500 2    50   Input ~ 0
@@
 F 0 "R35" V 7554 5350 50  0000 C CNN
 F 1 "2.2k" V 7645 5350 50  0000 C CNN
-F 2 "Resistor_SMD:R_0603_1608Metric" H 7750 5350 50  0001 C CNN
+F 2 "Resistor_SMD:R_0805_2012Metric" H 7750 5350 50  0001 C CNN
 F 3 "~" H 7750 5350 50  0001 C CNN
 	1    7750 5350
@@
 F 0 "R30" V 2093 2550 50  0000 C CNN
 F 1 "220" V 2184 2550 50  0000 C CNN
-F 2 "Resistor_SMD:R_0603_1608Metric" V 2230 2550 50  0001 C CNN
+F 2 "Resistor_SMD:R_0805_2012Metric" V 2230 2550 50  0001 C CNN
 F 3 "~" H 2300 2550 50  0001 C CNN
 	1    2300 2550
@@
 F 0 "C31" V 9500 5075 50  0000 C CNN
 F 1 "150nF" V 9575 5025 50  0000 C CNN
-F 2 "Capacitor_SMD:C_0603_1608Metric" H 9675 5000 50  0001 C CNN
+F 2 "Capacitor_SMD:C_0805_2012Metric" H 9675 5000 50  0001 C CNN
 F 3 "~" H 9675 5000 50  0001 C CNN
 	1    9675 5000
@@
 L power:+BATT #PWR0133
 U 1 1 5C2FECB9
-P 2750 3200
-F 0 "#PWR0133" H 2750 3050 50  0001 C CNN
-F 1 "+BATT" H 2765 3373 50  0000 C CNN
-F 2 "" H 2750 3200 50  0001 C CNN
-F 3 "" H 2750 3200 50  0001 C CNN
-	1    2750 3200
+P 2475 3100
+F 0 "#PWR0133" H 2475 2950 50  0001 C CNN
+F 1 "+BATT" H 2490 3273 50  0000 C CNN
+F 2 "" H 2475 3100 50  0001 C CNN
+F 3 "" H 2475 3100 50  0001 C CNN
+	1    2475 3100
 	1    0    0    -1
 $EndComp
@@
 L power:GND #PWR0134
 U 1 1 5C2FED50
-P 2150 4550
-F 0 "#PWR0134" H 2150 4300 50  0001 C CNN
-F 1 "GND" H 2155 4377 50  0000 C CNN
-F 2 "" H 2150 4550 50  0001 C CNN
-F 3 "" H 2150 4550 50  0001 C CNN
-	1    2150 4550
+P 2475 3900
+F 0 "#PWR0134" H 2475 3650 50  0001 C CNN
+F 1 "GND" H 2480 3727 50  0000 C CNN
+F 2 "" H 2475 3900 50  0001 C CNN
+F 3 "" H 2475 3900 50  0001 C CNN
+	1    2475 3900
 	1    0    0    -1
 $EndComp
@@
 Wire Wire Line
 	3125 4575 3200 4575
-Connection ~ 3125 3500
 Wire Wire Line
 	3125 3500 3200 3500
@@
 Wire Wire Line
 	6200 2450 5800 2450
-$Comp
-L Driver_LED:WS2811 U2
-U 1 1 5D266A84
-P 2150 4200
-F 0 "U2" H 1900 4650 50  0000 C CNN
-F 1 "WS2811" H 1900 4550 50  0000 C CNN
-F 2 "Package_SO:SSOP-8_3.95x5.21x3.27mm_P1.27mm" H 1850 4350 50  0001 C CNN
-F 3 "https://cdn-shop.adafruit.com/datasheets/WS2811.pdf" H 1950 4450 50  0001 C CNN
-	1    2150 4200
-	1    0    0    -1
-$EndComp
-Wire Wire Line
-	1550 4100 1750 4100
-Wire Wire Line
-	1750 4200 1625 4200
-Wire Wire Line
-	1625 4200 1625 3500
-Wire Wire Line
-	1625 3500 3125 3500
-Wire Wire Line
-	2150 4500 2150 4550
-$Comp
-L power:+BATT #PWR0145
-U 1 1 5D26BA5D
-P 2150 3825
-F 0 "#PWR0145" H 2150 3675 50  0001 C CNN
-F 1 "+BATT" H 2165 3998 50  0000 C CNN
-F 2 "" H 2150 3825 50  0001 C CNN
-F 3 "" H 2150 3825 50  0001 C CNN
-	1    2150 3825
-	1    0    0    -1
-$EndComp
-Wire Wire Line
-	2150 3825 2150 3900
-NoConn ~ 1750 4300
+Wire Wire Line
+	1875 3500 2075 3500
+$Comp
+L dk_Addressable-Specialty:COM-12999 D1
+U 1 1 5D2A09E9
+P 2575 3500
+F 0 "D1" H 2025 3900 60  0000 L CNN
+F 1 "COM-12999" H 2775 3025 60  0000 L CNN
+F 2 "digikey-footprints:LED_RGB_WP154A4SUREQBFZGC" H 2775 3700 60  0001 L CNN
+F 3 "https://cdn.sparkfun.com/datasheets/Components/LED/COM-12877.pdf" H 2775 3800 60  0001 L CNN
+F 4 "1568-1214-ND" H 2775 3900 60  0001 L CNN "Digi-Key_PN"
+F 5 "COM-12999" H 2775 4000 60  0001 L CNN "MPN"
+F 6 "Optoelectronics" H 2775 4100 60  0001 L CNN "Category"
+F 7 "Addressable, Specialty" H 2775 4200 60  0001 L CNN "Family"
+F 8 "https://cdn.sparkfun.com/datasheets/Components/LED/COM-12877.pdf" H 2775 4300 60  0001 L CNN "DK_Datasheet_Link"
+F 9 "/product-detail/en/sparkfun-electronics/COM-12999/1568-1214-ND/5673800" H 2775 4400 60  0001 L CNN "DK_Detail_Page"
+F 10 "ADDRESS LED DISC SER RGB 5MM 5PC" H 2775 4500 60  0001 L CNN "Description"
+F 11 "SparkFun Electronics" H 2775 4600 60  0001 L CNN "Manufacturer"
+F 12 "Active" H 2775 4700 60  0001 L CNN "Status"
+	1    2575 3500
+	1    0    0    -1
+$EndComp
+Wire Wire Line
+	2975 3500 3125 3500
+Connection ~ 3125 3500
 $EndSCHEMATC

Commit message: Began reworking sections
Parts:
- added J4: Conn_01x04_Male, MainBoard_Rev2:nav_switch_COM_08184, symbol Connector:Conn_01x04_Male
- D1: symbol dk_Addressable-Specialty:COM-12999 -> MainBoard-rescue:COM-12999-dk_Addressable-Specialty
Connections:
- net GND: now also J4.2 (Pin_2)
- new net BACK: J4.1 (Pin_1)
- new net DOWN: J4.4 (Pin_4)
- new net FWD: J4.3 (Pin_3)
Changed lines of the file:
@@
 	1875 3500 2075 3500
 $Comp
-L dk_Addressable-Specialty:COM-12999 D1
+L MainBoard-rescue:COM-12999-dk_Addressable-Specialty D1
 U 1 1 5D2A09E9
 P 2575 3500
+AR Path="/5D2A09E9" Ref="D1"  Part="1"
+AR Path="/5C2D6974/5D2A09E9" Ref="D1"  Part="1"
 F 0 "D1" H 2025 3900 60  0000 L CNN
 F 1 "COM-12999" H 2775 3025 60  0000 L CNN
@@
 	2975 3500 3125 3500
 Connection ~ 3125 3500
+$Comp
+L Connector:Conn_01x04_Male J4
+U 1 1 5D685BA0
+P 3800 6325
+F 0 "J4" H 3906 6603 50  0000 C CNN
+F 1 "Conn_01x04_Male" H 3906 6512 50  0000 C CNN
+F 2 "MainBoard_Rev2:nav_switch_COM_08184" H 3800 6325 50  0001 C CNN
+F 3 "~" H 3800 6325 50  0001 C CNN
+	1    3800 6325
+	1    0    0    -1
+$EndComp
+$Comp
+L power:GND #PWR0145
+U 1 1 5D6A22BA
+P 4250 6325
+F 0 "#PWR0145" H 4250 6075 50  0001 C CNN
+F 1 "GND" V 4255 6197 50  0000 R CNN
+F 2 "" H 4250 6325 50  0001 C CNN
+F 3 "" H 4250 6325 50  0001 C CNN
+	1    4250 6325
+	0    -1   -1   0
+$EndComp
+Wire Wire Line
+	4000 6325 4250 6325
+Text HLabel 4300 6225 2    50   Input ~ 0
+BACK
+Text HLabel 4300 6425 2    50   Input ~ 0
+FWD
+Text HLabel 4300 6525 2    50   Input ~ 0
+DOWN
+Wire Wire Line
+	4000 6225 4300 6225
+Wire Wire Line
+	4000 6425 4300 6425
+Wire Wire Line
+	4000 6525 4300 6525
 $EndSCHEMATC

Commit message: Continued work on the current electronics
Parts:
- C3: value 0.1uF -> 100nF
- C31: value 150nF -> 100nF
Changed lines of the file:
@@
 P 9675 5000
 F 0 "C31" V 9500 5075 50  0000 C CNN
-F 1 "150nF" V 9575 5025 50  0000 C CNN
+F 1 "100nF" V 9575 5025 50  0000 C CNN
 F 2 "Capacitor_SMD:C_0805_2012Metric" H 9675 5000 50  0001 C CNN
 F 3 "~" H 9675 5000 50  0001 C CNN
@@
 P 5750 1775
 F 0 "C3" H 5658 1729 50  0000 R CNN
-F 1 "0.1uF" H 5658 1820 50  0000 R CNN
+F 1 "100nF" H 5658 1820 50  0000 R CNN
 F 2 "Capacitor_SMD:C_0805_2012Metric" H 5750 1775 50  0001 C CNN
 F 3 "~" H 5750 1775 50  0001 C CNN
