File: Electronics/MainBoard_Rev2/Power.sch (KiCad schematic (older format))
At the start: 16 parts, among them U50 AP2114H-3_3TRG1, U51 LP3947

Commit message: Temporary polishing of PCB
Parts:
- removed R57: 100k, Resistor_SMD:R_0603_1608Metric, symbol Device:R_Small
- removed U51: LP3947, Package_SON:WSON-14-1EP_4.0x4.0mm_P0.5mm_EP2.6x2.6mm, symbol Battery_Management:LP3947
- added U4: MAX1555EZK_T, digikey-footprints:SOT-753, symbol dk_PMIC-Battery-Chargers:MAX1555EZK_T
- C50, C51, C52: footprint Capacitor_SMD:C_0603_1608Metric -> Capacitor_SMD:C_0805_2012Metric
- R52, R55: footprint Resistor_SMD:R_0603_1608Metric -> Resistor_SMD:R_0805_2012Metric
- R56: value 100k -> 200k; footprint Resistor_SMD:R_0603_1608Metric -> Resistor_SMD:R_0805_2012Metric
Connections:
- net labels added: CHG_Stat
- net labels removed: FastCHG_En, SCL, SDA
- wire segments 49 -> 46
- no-connect marks 5 -> 1
Changed lines of the file:
@@
 	4650 3350 4650 3100
-Wire Wire Line
-	3425 4650 3425 4500
 Wire Wire Line
 	4650 3650 4650 3750
@@
 L power:GND #PWR0107
 U 1 1 5C2BBAFA
-P 3425 4650
-F 0 "#PWR0107" H 3425 4400 50  0001 C CNN
-F 1 "GND" H 3430 4477 50  0000 C CNN
-F 2 "" H 3425 4650 50  0001 C CNN
-F 3 "" H 3425 4650 50  0001 C CNN
-	1    3425 4650
+P 3475 4050
+F 0 "#PWR0107" H 3475 3800 50  0001 C CNN
+F 1 "GND" H 3480 3877 50  0000 C CNN
+F 2 "" H 3475 4050 50  0001 C CNN
+F 3 "" H 3475 4050 50  0001 C CNN
+	1    3475 4050
 	1    0    0    -1
 $EndComp
@@
 F 0 "C52" H 7565 3146 50  0000 L CNN
 F 1 "10uF" H 7565 3055 50  0000 L CNN
-F 2 "Capacitor_SMD:C_0603_1608Metric" H 7488 2950 50  0001 C CNN
+F 2 "Capacitor_SMD:C_0805_2012Metric" H 7488 2950 50  0001 C CNN
 F 3 "~" H 7450 3100 50  0001 C CNN
 	1    7450 3100
@@
 F 0 "R52" H 4909 2696 50  0000 L CNN
 F 1 "10k" H 4909 2605 50  0000 L CNN
-F 2 "Resistor_SMD:R_0603_1608Metric" H 4850 2650 50  0001 C CNN
+F 2 "Resistor_SMD:R_0805_2012Metric" H 4850 2650 50  0001 C CNN
 F 3 "~" H 4850 2650 50  0001 C CNN
 	1    4850 2650
@@
 F 0 "C50" H 6015 3346 50  0000 L CNN
 F 1 "10uF" H 6015 3255 50  0000 L CNN
-F 2 "Capacitor_SMD:C_0603_1608Metric" H 5938 3150 50  0001 C CNN
+F 2 "Capacitor_SMD:C_0805_2012Metric" H 5938 3150 50  0001 C CNN
 F 3 "~" H 5900 3300 50  0001 C CNN
 	1    5900 3300
@@
 F 0 "R55" H 5859 4546 50  0000 L CNN
 F 1 "100k" H 5859 4455 50  0000 L CNN
-F 2 "Resistor_SMD:R_0603_1608Metric" H 5800 4500 50  0001 C CNN
+F 2 "Resistor_SMD:R_0805_2012Metric" H 5800 4500 50  0001 C CNN
 F 3 "~" H 5800 4500 50  0001 C CNN
 	1    5800 4500
@@
 P 5800 4700
 F 0 "R56" H 5859 4746 50  0000 L CNN
-F 1 "100k" H 5859 4655 50  0000 L CNN
-F 2 "Resistor_SMD:R_0603_1608Metric" H 5800 4700 50  0001 C CNN
+F 1 "200k" H 5859 4655 50  0000 L CNN
+F 2 "Resistor_SMD:R_0805_2012Metric" H 5800 4700 50  0001 C CNN
 F 3 "~" H 5800 4700 50  0001 C CNN
 	1    5800 4700
@@
 $EndComp
 $Comp
-L Device:R_Small R57
-U 1 1 5C2CC0A3
-P 5800 4900
-F 0 "R57" H 5859 4946 50  0000 L CNN
-F 1 "100k" H 5859 4855 50  0000 L CNN
-F 2 "Resistor_SMD:R_0603_1608Metric" H 5800 4900 50  0001 C CNN
-F 3 "~" H 5800 4900 50  0001 C CNN
-	1    5800 4900
-	1    0    0    -1
-$EndComp
-$Comp
 L power:GND #PWR0112
 U 1 1 5C2CC17A
-P 5800 5000
-F 0 "#PWR0112" H 5800 4750 50  0001 C CNN
-F 1 "GND" H 5805 4827 50  0000 C CNN
-F 2 "" H 5800 5000 50  0001 C CNN
-F 3 "" H 5800 5000 50  0001 C CNN
-	1    5800 5000
+P 5800 4800
+F 0 "#PWR0112" H 5800 4550 50  0001 C CNN
+F 1 "GND" H 5805 4627 50  0000 C CNN
+F 2 "" H 5800 4800 50  0001 C CNN
+F 3 "" H 5800 4800 50  0001 C CNN
+	1    5800 4800
 	1    0    0    -1
 $EndComp
@@
 B_Raw+
 Wire Wire Line
-	2925 3700 2850 3700
-Text HLabel 2850 3700 0    50   Input ~ 0
-FastCHG_En
-Wire Wire Line
 	6025 3100 5900 3100
 Connection ~ 5800 3100
@@
 F 0 "C51" H 6467 3346 50  0000 L CNN
 F 1 "150nF" H 6467 3255 50  0000 L CNN
-F 2 "Capacitor_SMD:C_0603_1608Metric" H 6375 3300 50  0001 C CNN
+F 2 "Capacitor_SMD:C_0805_2012Metric" H 6375 3300 50  0001 C CNN
 F 3 "~" H 6375 3300 50  0001 C CNN
 	1    6375 3300
@@
 	6375 2850 6450 2850
 Connection ~ 6375 3100
-Wire Wire Line
-	7350 2850 7350 2950
-Wire Wire Line
-	7450 2950 7350 2950
-Connection ~ 7450 2950
-Connection ~ 7350 2950
-$Comp
-L Battery_Management:LP3947 U51
-U 1 1 5D2733BC
-P 3525 3700
-F 0 "U51" H 3525 4578 50  0000 C CNN
-F 1 "LP3947" H 3200 4300 50  0000 C CNN
-F 2 "Package_SON:WSON-14-1EP_4.0x4.0mm_P0.5mm_EP2.6x2.6mm" H 4725 3050 50  0001 C CNN
-F 3 "http://www.ti.com/lit/ds/symlink/lp3947.pdf" H 3425 3900 50  0001 C CNN
-	1    3525 3700
-	1    0    0    -1
-$EndComp
 $Comp
 L Device:L_Core_Ferrite_Small L1
@@
 $EndComp
 Wire Wire Line
-	4125 3400 4125 3000
-NoConn ~ 4125 3900
-Wire Wire Line
-	3425 4500 3625 4500
-Wire Wire Line
-	3625 4500 3625 4400
-Connection ~ 3425 4500
-Wire Wire Line
-	3425 4500 3425 4400
-NoConn ~ 2925 3400
-NoConn ~ 2925 3500
-NoConn ~ 2925 3200
-Connection ~ 4125 3000
-Wire Wire Line
 	4125 3000 4225 3000
-Wire Wire Line
-	3625 3000 4125 3000
 $Comp
 L Device:C_Small C53
@@
 Wire Wire Line
 	3175 2625 3225 2625
-NoConn ~ 2925 3800
-Text GLabel 2825 4100 0    50   Input ~ 0
-SDA
-Text GLabel 2825 4000 0    50   Input ~ 0
-SCL
-Wire Wire Line
-	2825 4000 2925 4000
-Wire Wire Line
-	2825 4100 2925 4100
+Wire Wire Line
+	7350 2850 7450 2850
+Wire Wire Line
+	7450 2850 7450 2950
+Connection ~ 7450 2950
+NoConn ~ 7350 2950
+$Comp
+L dk_PMIC-Battery-Chargers:MAX1555EZK_T U4
+U 1 1 5D2797BC
+P 3575 3400
+F 0 "U4" H 3247 3453 60  0000 R CNN
+F 1 "MAX1555EZK_T" H 3247 3347 60  0000 R CNN
+F 2 "digikey-footprints:SOT-753" H 3775 3600 60  0001 L CNN
+F 3 "https://datasheets.maximintegrated.com/en/ds/MAX1551-MAX1555.pdf" H 3775 3700 60  0001 L CNN
+F 4 "MAX1555EZK+TCT-ND" H 3775 3800 60  0001 L CNN "Digi-Key_PN"
+F 5 "MAX1555EZK+T" H 3775 3900 60  0001 L CNN "MPN"
+F 6 "Integrated Circuits (ICs)" H 3775 4000 60  0001 L CNN "Category"
+F 7 "PMIC - Battery Chargers" H 3775 4100 60  0001 L CNN "Family"
+F 8 "https://datasheets.maximintegrated.com/en/ds/MAX1551-MAX1555.pdf" H 3775 4200 60  0001 L CNN "DK_Datasheet_Link"
+F 9 "/product-detail/en/maxim-integrated/MAX1555EZK-T/MAX1555EZK-TCT-ND/2699449" H 3775 4300 60  0001 L CNN "DK_Detail_Page"
+F 10 "IC BATT CHRGR LI+ 1CELL SOT23-5" H 3775 4400 60  0001 L CNN "Description"
+F 11 "Maxim Integrated" H 3775 4500 60  0001 L CNN "Manufacturer"
+F 12 "Active" H 3775 4600 60  0001 L CNN "Status"
+	1    3575 3400
+	1    0    0    -1
+$EndComp
+Wire Wire Line
+	3425 3000 3475 3000
+Wire Wire Line
+	3875 3500 4125 3500
+Wire Wire Line
+	4125 3000 4125 3500
+Wire Wire Line
+	3475 3800 3475 4050
+Text HLabel 4000 3750 3    50   Input ~ 0
+CHG_Stat
+Wire Wire Line
+	3875 3400 4000 3400
+Wire Wire Line
+	4000 3400 4000 3750
 $EndSCHEMATC

Commit message: Began reworking the PCB
Parts:
- added D?: D_Zener_ALT, Diode_SMD:D_SOD-123F, symbol Device:D_Zener_ALT
- added SW?: Rotary_Encoder, symbol Device:Rotary_Encoder
Connections:
- wire segments 46 -> 50
Changed lines of the file:
@@
 Wire Wire Line
 	4000 3400 4000 3750
+$Comp
+L Device:D_Zener_ALT D?
+U 1 1 5D685547
+P 7875 3225
+F 0 "D?" V 7829 3304 50  0000 L CNN
+F 1 "D_Zener_ALT" V 7920 3304 50  0000 L CNN
+F 2 "Diode_SMD:D_SOD-123F" H 7875 3225 50  0001 C CNN
+F 3 "~" H 7875 3225 50  0001 C CNN
+F 4 "F7701CT-ND" H 7875 3225 50  0001 C CNN "DigiKey"
+	1    7875 3225
+	0    1    1    0
+$EndComp
+Wire Wire Line
+	7450 3500 7875 3500
+Wire Wire Line
+	7875 3500 7875 3375
+Connection ~ 7450 3500
+Wire Wire Line
+	7600 2950 7875 2950
+Wire Wire Line
+	7875 2950 7875 3075
+Connection ~ 7600 2950
+$Comp
+L Device:Rotary_Encoder SW?
+U 1 1 5D688172
+P 9150 2900
+F 0 "SW?" H 9379 2946 50  0000 L CNN
+F 1 "Rotary_Encoder" H 9379 2855 50  0000 L CNN
+F 2 "" H 9000 3060 50  0001 C CNN
+F 3 "~" H 9150 3160 50  0001 C CNN
+	1    9150 2900
+	1    0    0    -1
+$EndComp
 $EndSCHEMATC

Commit message: Began reworking sections
Parts:
- removed C51: 150nF, Capacitor_SMD:C_0805_2012Metric, symbol Device:C_Small
- removed L1: 445-3654-1-ND, Inductor_SMD:L_1210_3225Metric, symbol Device:L_Core_Ferrite_Small
- removed SW?: Rotary_Encoder, symbol Device:Rotary_Encoder
- C50: value 10uF -> 1uF
- gave numbers to parts that had none: 1
Connections:
- wire segments 50 -> 46
- no-connect marks 1 -> 2
Other:
- moved on the sheet: C50, C52
Changed lines of the file:
@@
 L Device:C C52
 U 1 1 5C2BC1E8
-P 7450 3100
-F 0 "C52" H 7565 3146 50  0000 L CNN
-F 1 "10uF" H 7565 3055 50  0000 L CNN
-F 2 "Capacitor_SMD:C_0805_2012Metric" H 7488 2950 50  0001 C CNN
-F 3 "~" H 7450 3100 50  0001 C CNN
-	1    7450 3100
+P 7450 3250
+F 0 "C52" H 7565 3296 50  0000 L CNN
+F 1 "10uF" H 7565 3205 50  0000 L CNN
+F 2 "Capacitor_SMD:C_0805_2012Metric" H 7488 3100 50  0001 C CNN
+F 3 "~" H 7450 3250 50  0001 C CNN
+	1    7450 3250
 	1    0    0    -1
 $EndComp
 Wire Wire Line
 	7450 2950 7600 2950
-Wire Wire Line
-	7450 3250 7450 3500
-Wire Wire Line
-	7450 3500 6850 3500
 Connection ~ 6850 3500
 Wire Wire Line
@@
 L Device:C C50
 U 1 1 5C2CB5FD
-P 5900 3300
-F 0 "C50" H 6015 3346 50  0000 L CNN
-F 1 "10uF" H 6015 3255 50  0000 L CNN
-F 2 "Capacitor_SMD:C_0805_2012Metric" H 5938 3150 50  0001 C CNN
-F 3 "~" H 5900 3300 50  0001 C CNN
-	1    5900 3300
-	1    0    0    -1
-$EndComp
-Wire Wire Line
-	6375 3400 6375 3500
-Wire Wire Line
-	6375 3500 6850 3500
+P 6350 3300
+F 0 "C50" H 6465 3346 50  0000 L CNN
+F 1 "1uF" H 6465 3255 50  0000 L CNN
+F 2 "Capacitor_SMD:C_0805_2012Metric" H 6388 3150 50  0001 C CNN
+F 3 "~" H 6350 3300 50  0001 C CNN
+	1    6350 3300
+	1    0    0    -1
+$EndComp
 $Comp
 L Device:R_Small R55
@@
 Text Label 4575 3100 3    50   ~ 0
 B_Raw+
-Wire Wire Line
-	6025 3100 5900 3100
 Connection ~ 5800 3100
-$Comp
-L Device:C_Small C51
-U 1 1 5C2E8D17
-P 6375 3300
-F 0 "C51" H 6467 3346 50  0000 L CNN
-F 1 "150nF" H 6467 3255 50  0000 L CNN
-F 2 "Capacitor_SMD:C_0805_2012Metric" H 6375 3300 50  0001 C CNN
-F 3 "~" H 6375 3300 50  0001 C CNN
-	1    6375 3300
-	1    0    0    -1
-$EndComp
-Wire Wire Line
-	5900 3150 5900 3100
-Connection ~ 5900 3100
-Wire Wire Line
-	5900 3100 5800 3100
-Wire Wire Line
-	5900 3450 5900 3500
-Wire Wire Line
-	5900 3500 6375 3500
-Connection ~ 6375 3500
-Wire Wire Line
-	6225 3100 6375 3100
-Wire Wire Line
-	6375 3200 6375 3100
 Wire Wire Line
 	3425 2800 3425 3000
@@
 $EndComp
 Wire Wire Line
-	6375 3100 6375 2850
-Wire Wire Line
 	6375 2850 6450 2850
-Connection ~ 6375 3100
-$Comp
-L Device:L_Core_Ferrite_Small L1
-U 1 1 5D26A5A4
-P 6125 3100
-F 0 "L1" V 5947 3100 50  0000 C CNN
-F 1 "445-3654-1-ND" V 6038 3100 50  0000 C CNN
-F 2 "Inductor_SMD:L_1210_3225Metric" H 6125 3100 50  0001 C CNN
-F 3 "~" H 6125 3100 50  0001 C CNN
-	1    6125 3100
-	0    1    1    0
-$EndComp
 Wire Wire Line
 	4125 3000 4225 3000
@@
 Wire Wire Line
 	3175 2625 3225 2625
-Wire Wire Line
-	7350 2850 7450 2850
-Wire Wire Line
-	7450 2850 7450 2950
 Connection ~ 7450 2950
-NoConn ~ 7350 2950
 $Comp
 L dk_PMIC-Battery-Chargers:MAX1555EZK_T U4
@@
 	4000 3400 4000 3750
 $Comp
-L Device:D_Zener_ALT D?
+L Device:D_Zener_ALT D8
 U 1 1 5D685547
 P 7875 3225
-F 0 "D?" V 7829 3304 50  0000 L CNN
+F 0 "D8" V 7829 3304 50  0000 L CNN
 F 1 "D_Zener_ALT" V 7920 3304 50  0000 L CNN
 F 2 "Diode_SMD:D_SOD-123F" H 7875 3225 50  0001 C CNN
@@
 $EndComp
 Wire Wire Line
-	7450 3500 7875 3500
-Wire Wire Line
 	7875 3500 7875 3375
-Connection ~ 7450 3500
 Wire Wire Line
 	7600 2950 7875 2950
@@
 	7875 2950 7875 3075
 Connection ~ 7600 2950
-$Comp
-L Device:Rotary_Encoder SW?
-U 1 1 5D688172
-P 9150 2900
-F 0 "SW?" H 9379 2946 50  0000 L CNN
-F 1 "Rotary_Encoder" H 9379 2855 50  0000 L CNN
-F 2 "" H 9000 3060 50  0001 C CNN
-F 3 "~" H 9150 3160 50  0001 C CNN
-	1    9150 2900
-	1    0    0    -1
-$EndComp
+Wire Wire Line
+	6375 2850 6375 3100
+Wire Wire Line
+	6350 3500 6850 3500
+Wire Wire Line
+	5800 3100 6350 3100
+Wire Wire Line
+	6350 3100 6350 3150
+Connection ~ 6350 3100
+Wire Wire Line
+	6350 3100 6375 3100
+Wire Wire Line
+	6350 3450 6350 3500
+Wire Wire Line
+	6850 3500 7450 3500
+Wire Wire Line
+	7450 2950 7450 3100
+Wire Wire Line
+	7450 3400 7450 3500
+Connection ~ 7450 3500
+Wire Wire Line
+	7450 3500 7875 3500
+Wire Wire Line
+	7350 2950 7450 2950
+NoConn ~ 7350 2850
+NoConn ~ 3575 3000
 $EndSCHEMATC

Commit message: Last changes for a functional Lasertag, ordered!
Parts:
- D8: Digi-Key_PN (none) -> F7701CT-ND; DigiKey F7701CT-ND -> (none)
- DPWR1: Digi-Key_PN (none) -> CD0603-B0340RCT-ND
- QPWR1: Digi-Key IRLML6402PBFCT-ND -> (none); Digi-Key_PN (none) -> IRLML6402PBFCT-ND
- SWPWR1: Digi-Key_PN (none) -> CKN9565-ND
Changed lines of the file:
@@
 F 2 "Package_TO_SOT_SMD:SOT-23" H 5700 2925 50  0001 L CIN
 F 3 "https://www.infineon.com/dgdl/irlml6402pbf.pdf?fileId=5546d462533600a401535668d5c2263c" H 5500 3000 50  0001 L CNN
-F 4 "IRLML6402PBFCT-ND" V 5500 3000 50  0001 C CNN "Digi-Key"
+F 4 "IRLML6402PBFCT-ND" V 5500 3000 50  0001 C CNN "Digi-Key_PN"
 F 5 "IRLML6402TRPBF" V 5500 3000 50  0001 C CNN "MPN"
 	1    5500 3000
@@
 F 2 "Diode_SMD:D_0603_1608Metric" H 5650 2550 50  0001 C CNN
 F 3 "~" H 5650 2550 50  0001 C CNN
+F 4 "CD0603-B0340RCT-ND" H 5650 2550 50  0001 C CNN "Digi-Key_PN"
 	1    5650 2550
 	-1   0    0    1
@@
 F 2 "Connector_PinHeader_2.54mm:PinHeader_1x02_P2.54mm_Vertical" H 5000 3100 50  0001 C CNN
 F 3 "" H 5000 3100 50  0001 C CNN
+F 4 "CKN9565-ND" H 5000 3100 50  0001 C CNN "Digi-Key_PN"
 	1    5000 3100
 	1    0    0    -1
@@
 F 2 "Diode_SMD:D_SOD-123F" H 7875 3225 50  0001 C CNN
 F 3 "~" H 7875 3225 50  0001 C CNN
-F 4 "F7701CT-ND" H 7875 3225 50  0001 C CNN "DigiKey"
+F 4 "F7701CT-ND" H 7875 3225 50  0001 C CNN "Digi-Key_PN"
 	1    7875 3225
 	0    1    1    0

Commit message: Change a few names to use DigiKey Part Number
Parts:
- BT1: Digi-Key_PN (none) -> 455-1749-1-ND
Changed lines of the file:
@@
 F 4 "455-1749-1-ND" H 4650 3550 50  0001 C CNN "Digi-Key"
 F 5 "S2B-PH-SM4-TB(LF)(SN)" H 4650 3550 50  0001 C CNN "MPN"
+F 6 "455-1749-1-ND" H 4650 3550 50  0001 C CNN "Digi-Key_PN"
 	1    4650 3550
 	1    0    0    -1

Commit message: Modify board for the v3.3 release-ish
Parts:
- added C201: 0.1uF, Capacitor_SMD:C_0805_2012Metric, symbol Device:C_Small
- BT1: footprint Connector_JST:JST_PH_S2B-PH-SM4-TB_1x02-1MP_P2.00mm_Horizontal -> Connector_PinHeader_2.54mm:PinHeader_1x02_P2.54mm_Horizontal
- R55: value 100k -> 50k
- R56: value 200k -> 50k
Connections:
- net +3V3: now also U50.2 (VOUT)
- net B_Raw+: now also QPWR1.3 (D), SWPWR1.2 (B); no longer BT1.1 (+), C53.1, SWPWR1.1 (A), U4.5 (BAT)
- net GND: now also C201.2
- net V_SENSE: now also C201.1
- new net: BT1.1 (+), C53.1, SWPWR1.1 (A), U4.5 (BAT)
- no-connect marks 2 -> 1
Other:
- note added: "Higher tolerance resistors here!\n"
- moved on the sheet: C53
Changed lines of the file:
@@
 F 0 "BT1" H 4768 3646 50  0000 L CNN
 F 1 "Battery_Cell" H 4768 3555 50  0000 L CNN
-F 2 "Connector_JST:JST_PH_S2B-PH-SM4-TB_1x02-1MP_P2.00mm_Horizontal" V 4650 3610 50  0001 C CNN
+F 2 "Connector_PinHeader_2.54mm:PinHeader_1x02_P2.54mm_Horizontal" V 4650 3610 50  0001 C CNN
 F 3 "~" V 4650 3610 50  0001 C CNN
 F 4 "455-1749-1-ND" H 4650 3550 50  0001 C CNN "Digi-Key"
@@
 Wire Wire Line
 	6850 3600 6850 3500
-Wire Wire Line
-	4450 3000 4450 3100
-Wire Wire Line
-	4450 3100 4650 3100
 Text HLabel 3100 2800 0    50   Input ~ 0
 CHG_In
@@
 P 5800 4500
 F 0 "R55" H 5859 4546 50  0000 L CNN
-F 1 "100k" H 5859 4455 50  0000 L CNN
+F 1 "50k" H 5859 4455 50  0000 L CNN
 F 2 "Resistor_SMD:R_0805_2012Metric" H 5800 4500 50  0001 C CNN
 F 3 "~" H 5800 4500 50  0001 C CNN
@@
 P 5800 4700
 F 0 "R56" H 5859 4746 50  0000 L CNN
-F 1 "200k" H 5859 4655 50  0000 L CNN
+F 1 "50k" H 5859 4655 50  0000 L CNN
 F 2 "Resistor_SMD:R_0805_2012Metric" H 5800 4700 50  0001 C CNN
 F 3 "~" H 5800 4700 50  0001 C CNN
@@
 L power:GND #PWR0112
 U 1 1 5C2CC17A
-P 5800 4800
-F 0 "#PWR0112" H 5800 4550 50  0001 C CNN
-F 1 "GND" H 5805 4627 50  0000 C CNN
-F 2 "" H 5800 4800 50  0001 C CNN
-F 3 "" H 5800 4800 50  0001 C CNN
-	1    5800 4800
-	1    0    0    -1
-$EndComp
-Wire Wire Line
-	5800 4600 6250 4600
+P 5800 4850
+F 0 "#PWR0112" H 5800 4600 50  0001 C CNN
+F 1 "GND" H 5805 4677 50  0000 C CNN
+F 2 "" H 5800 4850 50  0001 C CNN
+F 3 "" H 5800 4850 50  0001 C CNN
+	1    5800 4850
+	1    0    0    -1
+$EndComp
+Wire Wire Line
+	5800 4600 6175 4600
 Connection ~ 5800 4600
 Text HLabel 6250 4600 2    50   Input ~ 0
@@
 Text Label 5800 4100 3    50   ~ 0
 B_Raw+
-Text Label 4575 3100 3    50   ~ 0
+Text Label 5275 3100 3    50   ~ 0
 B_Raw+
 Connection ~ 5800 3100
@@
 	1    0    0    -1
 $EndComp
-Wire Wire Line
-	6375 2850 6450 2850
-Wire Wire Line
-	4125 3000 4225 3000
 $Comp
 L Device:C_Small C53
 U 1 1 5D275BE8
-P 4225 3150
-F 0 "C53" H 4317 3196 50  0000 L CNN
-F 1 "10uF" H 4317 3105 50  0000 L CNN
-F 2 "Capacitor_SMD:C_0805_2012Metric" H 4225 3150 50  0001 C CNN
-F 3 "~" H 4225 3150 50  0001 C CNN
-	1    4225 3150
-	1    0    0    -1
-$EndComp
-Wire Wire Line
-	4225 3000 4225 3050
-Connection ~ 4225 3000
-Wire Wire Line
-	4225 3000 4450 3000
+P 4200 3600
+F 0 "C53" H 4292 3646 50  0000 L CNN
+F 1 "10uF" H 4292 3555 50  0000 L CNN
+F 2 "Capacitor_SMD:C_0805_2012Metric" H 4200 3600 50  0001 C CNN
+F 3 "~" H 4200 3600 50  0001 C CNN
+	1    4200 3600
+	1    0    0    -1
+$EndComp
 $Comp
 L power:GND #PWR0125
 U 1 1 5D2764A1
-P 4225 3250
-F 0 "#PWR0125" H 4225 3000 50  0001 C CNN
-F 1 "GND" H 4230 3077 50  0000 C CNN
-F 2 "" H 4225 3250 50  0001 C CNN
-F 3 "" H 4225 3250 50  0001 C CNN
-	1    4225 3250
+P 4200 3700
+F 0 "#PWR0125" H 4200 3450 50  0001 C CNN
+F 1 "GND" H 4205 3527 50  0000 C CNN
+F 2 "" H 4200 3700 50  0001 C CNN
+F 3 "" H 4200 3700 50  0001 C CNN
+	1    4200 3700
 	1    0    0    -1
 $EndComp
@@
 	3425 3000 3475 3000
 Wire Wire Line
-	3875 3500 4125 3500
-Wire Wire Line
-	4125 3000 4125 3500
-Wire Wire Line
 	3475 3800 3475 4050
 Text HLabel 4000 3750 3    50   Input ~ 0
@@
 Connection ~ 7600 2950
 Wire Wire Line
-	6375 2850 6375 3100
-Wire Wire Line
 	6350 3500 6850 3500
 Wire Wire Line
@@
 Wire Wire Line
 	6350 3100 6350 3150
-Connection ~ 6350 3100
-Wire Wire Line
-	6350 3100 6375 3100
 Wire Wire Line
 	6350 3450 6350 3500
@@
 Wire Wire Line
 	7350 2950 7450 2950
-NoConn ~ 7350 2850
 NoConn ~ 3575 3000
+Wire Notes Line
+	5650 4050 6075 4050
+Wire Notes Line
+	6075 4050 6075 5050
+Wire Notes Line
+	6075 5050 5650 5050
+Wire Notes Line
+	5650 5050 5650 4050
+Text Notes 5650 4050 0    50   ~ 0
+Higher tolerance resistors here!\n
+$Comp
+L Device:C_Small C201
+U 1 1 60D2EB62
+P 6175 4700
+F 0 "C201" H 6267 4746 50  0000 L CNN
+F 1 "0.1uF" H 6267 4655 50  0000 L CNN
+F 2 "Capacitor_SMD:C_0805_2012Metric" H 6175 4700 50  0001 C CNN
+F 3 "~" H 6175 4700 50  0001 C CNN
+	1    6175 4700
+	1    0    0    -1
+$EndComp
+Connection ~ 6175 4600
+Wire Wire Line
+	6175 4600 6250 4600
+Wire Wire Line
+	5800 4800 5800 4825
+Wire Wire Line
+	5800 4825 6175 4825
+Wire Wire Line
+	6175 4825 6175 4800
+Connection ~ 5800 4825
+Wire Wire Line
+	5800 4825 5800 4850
+Wire Wire Line
+	3875 3500 4200 3500
+Wire Wire Line
+	4200 3500 4200 3100
+Wire Wire Line
+	4200 3100 4650 3100
+Connection ~ 4200 3500
+Wire Wire Line
+	6350 2850 6350 3100
+Wire Wire Line
+	6350 2850 6450 2850
+Connection ~ 6350 3100
+Wire Wire Line
+	7350 2850 7350 2950
+Connection ~ 7350 2950
 $EndSCHEMATC
