File: Electronics/MainBoard_Rev2/USB_Connection.sch (KiCad schematic (older format))
At the start: 11 parts

Commit message: Rev 3.0 is now done!
Parts:
- C10, C11, CPRG1, CRST1: renamed from C?; footprint (none) -> Capacitor_SMD:C_0603_1608Metric
- DUSB1: renamed from D?; footprint (none) -> LED_SMD:LED_0603_1608Metric_Pad1.05x0.95mm_HandSolder
- J10: renamed from J?; footprint (none) -> Connector_USB:USB_Micro-B_Wuerth_629105150521
- R1, RRST1: renamed from R?; footprint (none) -> Resistor_SMD:R_0603_1608Metric
- SWPRG1: renamed from SWPRG; footprint (none) -> Button_Switch_SMD:Panasonic_EVQPUL_EVQPUC; Digi-Key (none) -> P10849SCT-ND
- SWRST1: renamed from SWRST; footprint (none) -> Button_Switch_SMD:Panasonic_EVQPUL_EVQPUC; Digi-Key (none) -> P10849SCT-ND
- gave numbers to parts that had none: 1
Other:
- note added: "Footprints!\n"
Changed lines of the file:
@@
 $EndDescr
 $Comp
-L Connector:USB_B_Micro J?
+L Connector:USB_B_Micro J10
 U 1 1 5C2BCA10
 P 3700 3850
-F 0 "J?" H 3755 4317 50  0000 C CNN
+F 0 "J10" H 3755 4317 50  0000 C CNN
 F 1 "USB_B_Micro" H 3755 4226 50  0000 C CNN
-F 2 "" H 3850 3800 50  0001 C CNN
+F 2 "Connector_USB:USB_Micro-B_Wuerth_629105150521" H 3850 3800 50  0001 C CNN
 F 3 "~" H 3850 3800 50  0001 C CNN
 	1    3700 3850
@@
 $EndComp
 $Comp
-L Interface_USB:FT230XS U?
+L Interface_USB:FT230XS U10
 U 1 1 5C2BCB35
 P 5450 3950
-F 0 "U?" H 5450 4828 50  0000 C CNN
+F 0 "U10" H 5450 4828 50  0000 C CNN
 F 1 "FT230XS" H 5450 4737 50  0000 C CNN
 F 2 "Package_SO:SSOP-16_3.9x4.9mm_P0.635mm" H 5900 3300 50  0001 C CNN
@@
 	4500 3850 4750 3850
 $Comp
-L power:GND #PWR?
+L power:GND #PWR0114
 U 1 1 5C2BCD0C
 P 3650 4400
-F 0 "#PWR?" H 3650 4150 50  0001 C CNN
+F 0 "#PWR0114" H 3650 4150 50  0001 C CNN
 F 1 "GND" H 3655 4227 50  0000 C CNN
 F 2 "" H 3650 4400 50  0001 C CNN
@@
 	5450 4650 5550 4650
 $Comp
-L power:GND #PWR?
+L power:GND #PWR0115
 U 1 1 5C2BCF34
 P 5450 4750
-F 0 "#PWR?" H 5450 4500 50  0001 C CNN
+F 0 "#PWR0115" H 5450 4500 50  0001 C CNN
 F 1 "GND" H 5455 4577 50  0000 C CNN
 F 2 "" H 5450 4750 50  0001 C CNN
@@
 	6700 3650 6150 3650
 $Comp
-L Device:C_Small C?
+L Device:C_Small C11
 U 1 1 5C2BD8B5
 P 4450 4250
-F 0 "C?" H 4358 4204 50  0000 R CNN
+F 0 "C11" H 4358 4204 50  0000 R CNN
 F 1 "150nF" H 4358 4295 50  0000 R CNN
-F 2 "" H 4450 4250 50  0001 C CNN
+F 2 "Capacitor_SMD:C_0603_1608Metric" H 4450 4250 50  0001 C CNN
 F 3 "~" H 4450 4250 50  0001 C CNN
 	1    4450 4250
@@
 Connection ~ 4700 4150
 $Comp
-L power:GND #PWR?
+L power:GND #PWR0116
 U 1 1 5C2BEFC1
 P 4450 4400
-F 0 "#PWR?" H 4450 4150 50  0001 C CNN
+F 0 "#PWR0116" H 4450 4150 50  0001 C CNN
 F 1 "GND" H 4455 4227 50  0000 C CNN
 F 2 "" H 4450 4400 50  0001 C CNN
@@
 	4450 4400 4450 4350
 $Comp
-L Device:C C?
+L Device:C C10
 U 1 1 5C2BF2BB
 P 4700 3100
-F 0 "C?" H 4815 3146 50  0000 L CNN
+F 0 "C10" H 4815 3146 50  0000 L CNN
 F 1 "10uF" H 4815 3055 50  0000 L CNN
-F 2 "" H 4738 2950 50  0001 C CNN
+F 2 "Capacitor_SMD:C_0603_1608Metric" H 4738 2950 50  0001 C CNN
 F 3 "~" H 4700 3100 50  0001 C CNN
 	1    4700 3100
@@
 	4700 3250 5350 3250
 $Comp
-L power:GND #PWR?
+L power:GND #PWR0117
 U 1 1 5C2BF368
 P 4700 2950
-F 0 "#PWR?" H 4700 2700 50  0001 C CNN
+F 0 "#PWR0117" H 4700 2700 50  0001 C CNN
 F 1 "GND" H 4705 2777 50  0000 C CNN
 F 2 "" H 4700 2950 50  0001 C CNN
@@
 $EndComp
 $Comp
-L Switch:SW_Push SWRST
+L Switch:SW_Push SWRST1
 U 1 1 5C2BF6AF
 P 5450 5450
-F 0 "SWRST" H 5450 5735 50  0000 C CNN
+F 0 "SWRST1" H 5450 5735 50  0000 C CNN
 F 1 "SW_Push" H 5450 5644 50  0000 C CNN
-F 2 "" H 5450 5650 50  0001 C CNN
+F 2 "Button_Switch_SMD:Panasonic_EVQPUL_EVQPUC" H 5450 5650 50  0001 C CNN
 F 3 "" H 5450 5650 50  0001 C CNN
+F 4 "P10849SCT-ND" H 5450 5450 50  0001 C CNN "Digi-Key"
 	1    5450 5450
 	1    0    0    -1
 $EndComp
 $Comp
-L Switch:SW_Push SWPRG
+L Switch:SW_Push SWPRG1
 U 1 1 5C2BF77A
 P 5450 5850
-F 0 "SWPRG" H 5450 6135 50  0000 C CNN
+F 0 "SWPRG1" H 5450 6135 50  0000 C CNN
 F 1 "SW_Push" H 5450 6044 50  0000 C CNN
-F 2 "" H 5450 6050 50  0001 C CNN
+F 2 "Button_Switch_SMD:Panasonic_EVQPUL_EVQPUC" H 5450 6050 50  0001 C CNN
 F 3 "" H 5450 6050 50  0001 C CNN
+F 4 "P10849SCT-ND" H 5450 5850 50  0001 C CNN "Digi-Key"
 	1    5450 5850
 	1    0    0    -1
@@
 	5150 5850 5150 6000
 $Comp
-L power:GND #PWR?
+L power:GND #PWR0118
 U 1 1 5C2C0152
 P 5150 6000
-F 0 "#PWR?" H 5150 5750 50  0001 C CNN
+F 0 "#PWR0118" H 5150 5750 50  0001 C CNN
 F 1 "GND" H 5155 5827 50  0000 C CNN
 F 2 "" H 5150 6000 50  0001 C CNN
@@
 	5650 5850 5950 5850
 $Comp
-L Device:C_Small C?
+L Device:C_Small CRST1
 U 1 1 5C2C09DB
 P 5950 5550
-F 0 "C?" H 6042 5596 50  0000 L CNN
+F 0 "CRST1" H 6042 5596 50  0000 L CNN
 F 1 "150nF" H 6042 5505 50  0000 L CNN
-F 2 "" H 5950 5550 50  0001 C CNN
+F 2 "Capacitor_SMD:C_0603_1608Metric" H 5950 5550 50  0001 C CNN
 F 3 "~" H 5950 5550 50  0001 C CNN
 	1    5950 5550
@@
 	5950 5450 6450 5450
 $Comp
-L Device:C_Small C?
+L Device:C_Small CPRG1
 U 1 1 5C2C0A50
 P 5950 5950
-F 0 "C?" H 6042 5996 50  0000 L CNN
+F 0 "CPRG1" H 6042 5996 50  0000 L CNN
 F 1 "150nF" H 6042 5905 50  0000 L CNN
-F 2 "" H 5950 5950 50  0001 C CNN
+F 2 "Capacitor_SMD:C_0603_1608Metric" H 5950 5950 50  0001 C CNN
 F 3 "~" H 5950 5950 50  0001 C CNN
 	1    5950 5950
@@
 	5850 6050 5850 6150
 $Comp
-L power:GND #PWR?
+L power:GND #PWR0119
 U 1 1 5C2C15E8
 P 5850 6150
-F 0 "#PWR?" H 5850 5900 50  0001 C CNN
+F 0 "#PWR0119" H 5850 5900 50  0001 C CNN
 F 1 "GND" H 5855 5977 50  0000 C CNN
 F 2 "" H 5850 6150 50  0001 C CNN
@@
 $EndComp
 $Comp
-L Device:R_Small R?
+L Device:R_Small RRST1
 U 1 1 5C2C173B
 P 5950 5350
-F 0 "R?" H 6009 5396 50  0000 L CNN
+F 0 "RRST1" H 6009 5396 50  0000 L CNN
 F 1 "R_Small" H 6009 5305 50  0000 L CNN
-F 2 "" H 5950 5350 50  0001 C CNN
+F 2 "Resistor_SMD:R_0603_1608Metric" H 5950 5350 50  0001 C CNN
 F 3 "~" H 5950 5350 50  0001 C CNN
 	1    5950 5350
@@
 $EndComp
 $Comp
-L power:+3.3V #PWR?
+L power:+3.3V #PWR0120
 U 1 1 5C2C17A7
 P 5950 5250
-F 0 "#PWR?" H 5950 5100 50  0001 C CNN
+F 0 "#PWR0120" H 5950 5100 50  0001 C CNN
 F 1 "+3.3V" H 5965 5423 50  0000 C CNN
 F 2 "" H 5950 5250 50  0001 C CNN
@@
 	6150 4050 6350 4050
 $Comp
-L Device:LED D?
+L Device:LED DUSB1
 U 1 1 5C2DA5D6
 P 6600 4375
-F 0 "D?" H 6591 4591 50  0000 C CNN
+F 0 "DUSB1" H 6591 4591 50  0000 C CNN
 F 1 "LED" H 6591 4500 50  0000 C CNN
-F 2 "" H 6600 4375 50  0001 C CNN
+F 2 "LED_SMD:LED_0603_1608Metric_Pad1.05x0.95mm_HandSolder" H 6600 4375 50  0001 C CNN
 F 3 "~" H 6600 4375 50  0001 C CNN
 	1    6600 4375
@@
 	6450 4150 6150 4150
 $Comp
-L Device:R_Small R?
+L Device:R_Small R1
 U 1 1 5C2DC6E6
 P 6875 4375
-F 0 "R?" V 6679 4375 50  0000 C CNN
+F 0 "R1" V 6679 4375 50  0000 C CNN
 F 1 "2.2k" V 6770 4375 50  0000 C CNN
-F 2 "" H 6875 4375 50  0001 C CNN
+F 2 "Resistor_SMD:R_0603_1608Metric" H 6875 4375 50  0001 C CNN
 F 3 "~" H 6875 4375 50  0001 C CNN
 	1    6875 4375
@@
 Text Label 7250 4375 2    50   ~ 0
 USB3.3
+Text Notes 5125 5900 1    50   ~ 0
+Footprints!\n
 $EndSCHEMATC

Commit message: Adjusted a few resistor values, added I2S pinout
Parts:
- removed CPRG1: 150nF, Capacitor_SMD:C_0603_1608Metric, symbol Device:C_Small
- R1: value 2.2k -> 220
Connections:
- wire segments 44 -> 41
Changed lines of the file:
@@
 Wire Wire Line
 	5650 5450 5950 5450
-Wire Wire Line
-	5650 5850 5950 5850
 $Comp
 L Device:C_Small CRST1
@@
 Wire Wire Line
 	5950 5450 6450 5450
-$Comp
-L Device:C_Small CPRG1
-U 1 1 5C2C0A50
-P 5950 5950
-F 0 "CPRG1" H 6042 5996 50  0000 L CNN
-F 1 "150nF" H 6042 5905 50  0000 L CNN
-F 2 "Capacitor_SMD:C_0603_1608Metric" H 5950 5950 50  0001 C CNN
-F 3 "~" H 5950 5950 50  0001 C CNN
-	1    5950 5950
-	1    0    0    -1
-$EndComp
-Connection ~ 5950 5850
-Wire Wire Line
-	5950 5850 6450 5850
 Wire Wire Line
 	5950 5650 5850 5650
-Wire Wire Line
-	5850 5650 5850 6050
-Wire Wire Line
-	5950 6050 5850 6050
-Connection ~ 5850 6050
-Wire Wire Line
-	5850 6050 5850 6150
 $Comp
 L power:GND #PWR0119
@@
 P 6875 4375
 F 0 "R1" V 6679 4375 50  0000 C CNN
-F 1 "2.2k" V 6770 4375 50  0000 C CNN
+F 1 "220" V 6770 4375 50  0000 C CNN
 F 2 "Resistor_SMD:R_0603_1608Metric" H 6875 4375 50  0001 C CNN
 F 3 "~" H 6875 4375 50  0001 C CNN
@@
 Text Notes 5125 5900 1    50   ~ 0
 Footprints!\n
+Wire Wire Line
+	5650 5850 6450 5850
+Wire Wire Line
+	5850 5650 5850 6150
 $EndSCHEMATC

Commit message: MORE
Parts:
- removed CRST1: 150nF, Capacitor_SMD:C_0603_1608Metric, symbol Device:C_Small
- removed RRST1: R_Small, Resistor_SMD:R_0603_1608Metric, symbol Device:R_Small
- removed SWPRG1, SWRST1: SW_Push, Button_Switch_SMD:Panasonic_EVQPUL_EVQPUC, symbol Switch:SW_Push
- removed U10: FT230XS, Package_SO:SSOP-16_3.9x4.9mm_P0.635mm, symbol Interface_USB:FT230XS
- added C19: 100nF, Capacitor_SMD:C_0805_2012Metric, symbol Device:C_Small
- added Q5, Q6: Q_NPN_BEC, Package_TO_SOT_SMD:SOT-23, symbol Device:Q_NPN_BEC
- added R13, R14, R15: R_Small, Resistor_SMD:R_0805_2012Metric, symbol Device:R_Small
- added U13: FT231XS, Package_SO:SSOP-20_3.9x8.7mm_P0.635mm, symbol Interface_USB:FT231XS
- C8: renamed from C11; footprint Capacitor_SMD:C_0603_1608Metric -> Capacitor_SMD:C_0805_2012Metric
- C9: renamed from C10; footprint Capacitor_SMD:C_0603_1608Metric -> Capacitor_SMD:C_0805_2012Metric
- DUSB1: footprint LED_SMD:LED_0603_1608Metric_Pad1.05x0.95mm_HandSolder -> LED_SMD:LED_0805_2012Metric
- R12: renamed from R1; footprint Resistor_SMD:R_0603_1608Metric -> Resistor_SMD:R_0805_2012Metric
- renumbered J10 to J3
Connections:
- wire segments 41 -> 50
Other:
- note removed: "Footprints!\n"
- moved on the sheet: DUSB1, R12

Commit message: Continued work on the current electronics
Parts:
- C8: value 150nF -> 100nF
- R13, R14: value R_Small -> 10k
Changed lines of the file:
@@
 P 4450 4250
 F 0 "C8" H 4358 4204 50  0000 R CNN
-F 1 "150nF" H 4358 4295 50  0000 R CNN
+F 1 "100nF" H 4358 4295 50  0000 R CNN
 F 2 "Capacitor_SMD:C_0805_2012Metric" H 4450 4250 50  0001 C CNN
 F 3 "~" H 4450 4250 50  0001 C CNN
@@
 P 7100 3850
 F 0 "R13" V 6904 3850 50  0000 C CNN
-F 1 "R_Small" V 6995 3850 50  0000 C CNN
+F 1 "10k" V 6995 3850 50  0000 C CNN
 F 2 "Resistor_SMD:R_0805_2012Metric" H 7100 3850 50  0001 C CNN
 F 3 "~" H 7100 3850 50  0001 C CNN
@@
 P 7100 4350
 F 0 "R14" V 6904 4350 50  0000 C CNN
-F 1 "R_Small" V 6995 4350 50  0000 C CNN
+F 1 "10k" V 6995 4350 50  0000 C CNN
 F 2 "Resistor_SMD:R_0805_2012Metric" H 7100 4350 50  0001 C CNN
 F 3 "~" H 7100 4350 50  0001 C CNN

Commit message: Last changes for a functional Lasertag, ordered!
Parts:
- J3: Digi-Key_PN (none) -> 732-5960-1-ND
- U13: Digi-Key_PN (none) -> 768-1129-1-ND
Changed lines of the file:
@@
 F 2 "Connector_USB:USB_Micro-B_Wuerth_629105150521" H 3850 3800 50  0001 C CNN
 F 3 "~" H 3850 3800 50  0001 C CNN
+F 4 "732-5960-1-ND" H 3700 3850 50  0001 C CNN "Digi-Key_PN"
 	1    3700 3850
 	1    0    0    -1
@@
 F 2 "Package_SO:SSOP-20_3.9x8.7mm_P0.635mm" H 6050 3200 50  0001 C CNN
 F 3 "http://www.ftdichip.com/Products/ICs/FT231X.html" H 5450 4150 50  0001 C CNN
+F 4 "768-1129-1-ND" H 5450 4150 50  0001 C CNN "Digi-Key_PN"
 	1    5450 4150
 	1    0    0    -1

Commit message: Change a few names to use DigiKey Part Number
Parts:
- Q5, Q6: Digi-Key_PN (none) -> 1727-2956-1-ND
Changed lines of the file:
@@
 F 2 "Package_TO_SOT_SMD:SOT-23" H 7600 3950 50  0001 C CNN
 F 3 "~" H 7400 3850 50  0001 C CNN
+F 4 "1727-2956-1-ND" H 7400 3850 50  0001 C CNN "Digi-Key_PN"
 	1    7400 3850
 	1    0    0    -1
@@
 F 2 "Package_TO_SOT_SMD:SOT-23" H 7600 4450 50  0001 C CNN
 F 3 "~" H 7400 4350 50  0001 C CNN
+F 4 "1727-2956-1-ND" H 7400 4350 50  0001 C CNN "Digi-Key_PN"
 	1    7400 4350
 	1    0    0    -1

Commit message: Modify board for the v3.3 release-ish
Parts:
- J3: symbol Connector:USB_B_Micro -> MainBoard-rescue:USB_B_Micro-Connector
- U13: symbol Interface_USB:FT231XS -> MainBoard-rescue:FT231XS-Interface_USB
Changed lines of the file:
@@
 $EndDescr
 $Comp
-L Connector:USB_B_Micro J3
+L MainBoard-rescue:USB_B_Micro-Connector J3
 U 1 1 5C2BCA10
 P 3700 3850
+AR Path="/5C2BCA10" Ref="J3"  Part="1"
+AR Path="/5C2BC95D/5C2BCA10" Ref="J3"  Part="1"
 F 0 "J3" H 3755 4317 50  0000 C CNN
 F 1 "USB_B_Micro" H 3755 4226 50  0000 C CNN
@@
 USB3.3
 $Comp
-L Interface_USB:FT231XS U13
+L MainBoard-rescue:FT231XS-Interface_USB U13
 U 1 1 5C7F8FA0
 P 5450 4150
+AR Path="/5C7F8FA0" Ref="U13"  Part="1"
+AR Path="/5C2BC95D/5C7F8FA0" Ref="U13"  Part="1"
 F 0 "U13" H 5450 5228 50  0000 C CNN
 F 1 "FT231XS" H 5450 5137 50  0000 C CNN
